File: kicad/ELSONIC/POWER_BD_NV2/POWER_BD_NV2.kicad_sch (KiCad schematic)
At the start: 76 parts, among them J1 SMW250-02P, J2 SMW250-06P, J3 TAP_250, J5 TAP_250, T1 220V/9V, U1 ICE3BR0665J, U2 PC817, U3 LM7805_TO220, U4 H11AA1, U5 ATTINY85-20PU_1

Commit message: POWER_BD_NV2: PCB/회로도 업데이트 및 거버 파일 추가
Parts:
- removed C6: EC47uF/35V, symbol 04_MyLib_Passive:C_Pol
- removed D1: GBJ406, GBL406BPC01HF, symbol 03_MyLib_Active:GBL406
- removed F1: SR5/2.5A, SR525ABK, symbol 05_MyLib_Device:SR525A
- removed T1: 220V/9V, symbol 04_MyLib_Passive:Transformer_1P_1S
- removed U4: H11AA1, DIP762W50P254L730H410Q6, symbol 01_MyLib_ICs:H11AA1
- removed VR1: TL431ILPR, 03_MyFoot_Active:TO92250P470H770-3, symbol 01_MyLib_ICs:TL431ILPR
- added A1, ACL2, ACN2, G1: TAP_250, 02_MyFoot_Connectors:TAP_250, symbol 02_MyLib_Connectors:TAP_250
- added C10: EC47uF/35V, 04_MyFoot_Passive:CP_Radial_D5.0mm_P2.00mm, symbol 04_MyLib_Passive:C_Pol
- added C11, C13: MLCC475, 04_MyFoot_Passive:C_Disc_D6.0mm_P5.00mm, symbol 04_MyLib_Passive:C
- added C31: MPP104/600V, 04_MyFoot_Passive:C_PP_L23.0mm_W10.9mm_P21.2mm, symbol 04_MyLib_Passive:C
- added C32, C33: CR1201, 04_MyFoot_Passive:SPARK_KILLER, symbol 04_MyLib_Passive:CR1201
- added D1: GBJ406, 03_MyFoot_Active:GBJ406, symbol 03_MyLib_Active:GBJ406
- added F2: SR5/2.5A, 05_MyFoot_Others:SR525ABK, symbol 05_MyLib_Others:SR525A
- added H2, H3: GND, 06_MyFoot_Mechanical:MTHole_3.5mm_7.5mmPad_GND, symbol Mechanical:MountingHole_Pad
- added H4: MountingHole, 06_MyFoot_Mechanical:MTHole_3.5mm, symbol 06_MyLib_Mechanical:MountingHole
- added LED2: RED/3Pi, 03_MyFoot_Active:LED_D3.0mm, symbol 03_MyLib_Active:LED
- added R10: 3.3K, 04_MyFoot_Passive:R_Axial_0.25W_P10.16mm, symbol 04_MyLib_Passive:R
- added R21: 1K, 04_MyFoot_Passive:R_Axial_0.25W_P10.16mm, symbol 04_MyLib_Passive:R
- added R23: 330R, 04_MyFoot_Passive:R_Axial_0.25W_P10.16mm, symbol 04_MyLib_Passive:R
- added R24: 220R/1W, 04_MyFoot_Passive:R_Axial_1W_P14.6mm, symbol 04_MyLib_Passive:R
- added R25: 2K/1W, 04_MyFoot_Passive:R_Axial_1W_P14.6mm, symbol 04_MyLib_Passive:R
- added R26: 100K/NOT, 04_MyFoot_Passive:R_Axial_0.25W_P10.16mm, symbol 04_MyLib_Passive:R
- added R9: 4.7K, 04_MyFoot_Passive:R_Axial_0.25W_P10.16mm, symbol 04_MyLib_Passive:R
- added T1: EI2811BP, 04_MyFoot_Passive:EI2811BP, symbol 04_MyLib_Passive:EI2811BP
- added U2: H11AA1, 01_MyFoot_ICs:DIP-6_W7.62mm, symbol 01_MyLib_ICs:H11AA1
- added U5: MOC3021M, 01_MyFoot_ICs:DIP-6_W7.62mm, symbol 01_MyLib_ICs:MOC3021M
- added VR1: TL431A, 01_MyFoot_ICs:TO92_P2.5mm, symbol 01_MyLib_ICs:TL431A
- A2: renamed from J5; footprint (none) -> 02_MyFoot_Connectors:TAP_250
- ACL1: renamed from L1; footprint (none) -> 02_MyFoot_Connectors:TAP_250
- ACN1: renamed from N1; footprint (none) -> 02_MyFoot_Connectors:TAP_250
- C1: renamed from C3; footprint (none) -> 04_MyFoot_Passive:DS222M
- C12: renamed from C28; footprint (none) -> 04_MyFoot_Passive:C_Disc_D4.7mm_T3.0mm_P5.00mm
- C14: renamed from C7; footprint (none) -> 04_MyFoot_Passive:DS222M
- C15: renamed from C11; footprint (none) -> 04_MyFoot_Passive:C_Disc_D4.7mm_P5.00mm
- C16: renamed from C15; footprint (none) -> 04_MyFoot_Passive:C_Disc_D4.7mm_P5.00mm
- C17: renamed from C14; footprint (none) -> 04_MyFoot_Passive:C_Disc_D4.7mm_P5.00mm
- C18: renamed from C13; footprint (none) -> 04_MyFoot_Passive:C_Disc_D4.7mm_P5.00mm
- C19: renamed from C12; value MLCC102 -> MLCC224; footprint (none) -> 04_MyFoot_Passive:C_Disc_D4.7mm_P5.00mm
- C2: footprint (none) -> 04_MyFoot_Passive:DS222M
- C20: renamed from C18; footprint (none) -> 04_MyFoot_Passive:CP_Radial_D12.5mm_P5.00mm
- C21: renamed from C17; footprint (none) -> 04_MyFoot_Passive:CP_Radial_D10.0mm_P5.00mm
- C22: renamed from C16; footprint (none) -> 04_MyFoot_Passive:CP_Radial_D10.0mm_P5.00mm
- C23: renamed from C19; footprint (none) -> 04_MyFoot_Passive:CP_Radial_D10.0mm_P5.00mm
- C24: renamed from C20; footprint (none) -> 04_MyFoot_Passive:CP_Radial_D10.0mm_P5.00mm
- C25: renamed from C21; footprint (none) -> 04_MyFoot_Passive:CP_Radial_D10.0mm_P5.00mm
- C26: renamed from C22; footprint (none) -> 04_MyFoot_Passive:C_Disc_D4.7mm_T3.0mm_P5.00mm
- C27: renamed from C23; footprint (none) -> 04_MyFoot_Passive:C_Disc_D4.7mm_T3.0mm_P5.00mm
- C28: renamed from C24; footprint (none) -> 04_MyFoot_Passive:C_Disc_D4.7mm_T3.0mm_P5.00mm
- C29: renamed from C26; footprint (none) -> 04_MyFoot_Passive:CP_Radial_D6.3mm_P2.50mm
- C3: renamed from C1; value CR1201 -> MP104K/275V; footprint (none) -> 04_MyFoot_Passive:104K_275V
- C30: renamed from C25; footprint (none) -> 04_MyFoot_Passive:C_Disc_D4.7mm_T3.0mm_P5.00mm
- C4: footprint (none) -> 04_MyFoot_Passive:82uF_400V
- C5: renamed from C8; footprint (none) -> 04_MyFoot_Passive:C_Disc_D4.7mm_T3.0mm_P5.00mm
- C6: renamed from C9; footprint (none) -> 04_MyFoot_Passive:C_Disc_D4.7mm_P5.00mm
- C7: renamed from C5; footprint (none) -> 04_MyFoot_Passive:C_Disc_D6.0mm_P5.00mm
- C8: renamed from C27; footprint (none) -> 04_MyFoot_Passive:C_Disc_D4.7mm_P5.00mm
- C9: renamed from C10; footprint (none) -> 04_MyFoot_Passive:C_Disc_D4.7mm_T3.0mm_P5.00mm
- D2: renamed from D6; footprint Diode_THT:D_DO-41_SOD81_P10.16mm_Horizontal -> 03_MyFoot_Active:Diode_P10.16mm
- D3: renamed from D4; footprint Diode_THT:D_DO-41_SOD81_P10.16mm_Horizontal -> 03_MyFoot_Active:Diode_P10.16mm
- D5: renamed from D7; footprint 03_MyFoot_Active:TO255P510X1070X2140-3P -> 03_MyFoot_Active:TO220AB_P2.55mm
- D6: renamed from D5; footprint 03_MyFoot_Active:TO255P510X1070X2140-3P -> 03_MyFoot_Active:TO220AB_P2.55mm
- D7: renamed from D3; footprint 03_MyFoot_Active:TO255P510X1070X2140-3P -> 03_MyFoot_Active:TO220AB_P2.55mm
- FG1: renamed from J3; footprint (none) -> 02_MyFoot_Connectors:TAP_250
- H1: renamed from H3; footprint (none) -> 06_MyFoot_Mechanical:MTHole_3.5mm_7.5mmPad_GND
- J2: footprint 02_MyFoot_Connectors:SMW25006 -> 02_MyFoot_Connectors:SMW250_06P
- J3: renamed from J1; footprint 02_MyFoot_Connectors:SMW25002 -> 02_MyFoot_Connectors:SMW250_02P
- L1: renamed from L4; footprint (none) -> 04_MyFoot_Passive:L_Radial_D7.5mm_P3.50mm
- L2, L3: footprint (none) -> 04_MyFoot_Passive:L_Radial_D7.5mm_P3.50mm
- LED1: footprint (none) -> 03_MyFoot_Active:LED_D3.0mm
- LF1: footprint (none) -> 04_MyFoot_Passive:LF1140
- R1: footprint (none) -> 04_MyFoot_Passive:R_Axial_1W_P14.6mm
- R11: renamed from R19; footprint 04_MyFoot_Passive:R_Axial_P10.16mm -> 04_MyFoot_Passive:R_Axial_0.25W_P10.16mm
- R12: renamed from R7; footprint (none) -> 04_MyFoot_Passive:R_Axial_0.25W_P10.16mm
- R13: renamed from R8; footprint (none) -> 04_MyFoot_Passive:R_Axial_0.25W_P10.16mm
- R14: renamed from R15; value 10R/1W -> 10R; footprint 04_MyFoot_Passive:R_Axial_P10.16mm -> 04_MyFoot_Passive:R_Axial_0.25W_P10.16mm
- R15: renamed from R14; value 10R/1W -> 10R; footprint 04_MyFoot_Passive:R_Axial_P10.16mm -> 04_MyFoot_Passive:R_Axial_0.25W_P10.16mm
- R16: renamed from R13; value 10R/1W -> 10R; footprint 04_MyFoot_Passive:R_Axial_P10.16mm -> 04_MyFoot_Passive:R_Axial_0.25W_P10.16mm
- R17: renamed from R10; value 12K -> 68K; footprint 04_MyFoot_Passive:R_Axial_P10.16mm -> 04_MyFoot_Passive:R_Axial_0.25W_P10.16mm
- R18: renamed from R12; value 10K -> 20K; footprint 04_MyFoot_Passive:R_Axial_P10.16mm -> 04_MyFoot_Passive:R_Axial_0.25W_P10.16mm
- R19: renamed from R11; value 220R -> 18K; footprint 04_MyFoot_Passive:R_Axial_P10.16mm -> 04_MyFoot_Passive:R_Axial_0.25W_P10.16mm
- R2: renamed from R17; footprint (none) -> 04_MyFoot_Passive:R_Axial_0.25W_P10.16mm
- R20: renamed from R9; value 1.2K -> 10K; footprint 04_MyFoot_Passive:R_Axial_P10.16mm -> 04_MyFoot_Passive:R_Axial_0.25W_P10.16mm
- R22: renamed from R16; footprint 04_MyFoot_Passive:R_Axial_P10.16mm -> 04_MyFoot_Passive:R_Axial_0.25W_P10.16mm
- R3: renamed from R4; footprint (none) -> 04_MyFoot_Passive:R_Axial_1W_P14.6mm
- R4: renamed from R3; footprint (none) -> 04_MyFoot_Passive:R_Axial_1W_P14.6mm
- R5: renamed from R2; footprint (none) -> 04_MyFoot_Passive:R_Axial_2W_P20.32mm
- R6: renamed from R18; footprint 04_MyFoot_Passive:R_Axial_P10.16mm -> 04_MyFoot_Passive:R_Axial_0.25W_P10.16mm
- R7: renamed from R5; footprint (none) -> 04_MyFoot_Passive:R_Axial_0.25W_P10.16mm
- R8: renamed from R6; footprint (none) -> 04_MyFoot_Passive:R_Axial_0.25W_P10.16mm
- RV1: footprint MOV14D471K -> 04_MyFoot_Passive:TNR14D_P7.62
- T2: renamed from TR1; footprint (none) -> 04_MyFoot_Passive:EER28_35_12P
- U1: footprint DIP788W56P254L944H480Q8N -> 01_MyFoot_ICs:DIP-8_W7.62mm_Socket
- U3: renamed from U2; footprint DIP762W50P254L495H455Q4 -> 01_MyFoot_ICs:DIP-4_W7.62mm_Socket
- U4: renamed from U5; footprint 8P3_ATM -> 01_MyFoot_ICs:DIP-8_W7.62mm_Socket
- U6: renamed from U3; footprint Package_TO_SOT_THT:TO-220-3_Vertical -> 01_MyFoot_ICs:TO220_P2.54mm
- renumbered D2 to D4
Connections:
- net +5V: now also U4.8 (VCC), R9.2
- net Earth: now also C10.2, D1.4 (-)
- net GND: now also R20.1, U4.4 (GND), C11.1, C13.1, H2.1, H3.1, LED2.1 (K), U2.4, U5.2, VR1.2
- net L01: now also RV1.2, ACL2.1 (Pin_1), ACL2.2 (Pin_2), C33.1, T1.2 (AB); no longer RV1.1
- net N01: now also RV1.1, A1.1 (Pin_1), A1.2 (Pin_2), C31.2, C32.1, C33.2, F2.1, R26.2, T1.1 (AA)
- net PWM_PW: now also C11.2, R10.1, R9.1
- net ZVC: now also U2.5
- net at D3.1 (K), R7.1: now also C10.1
- net at C19.2, R19.1, R20.2: now also VR1.1
- net at C2.2, LF1.2, R1.2: now also F2.2; no longer RV1.2
- net at R2.1: now also T1.4 (SB)
- net at R2.2: now also U2.1
- net at C15.1, R12.2, R13.1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: now also VR1.3
- net at A2.1 (Pin_1): now also A2.2 (Pin_2), ACN2.1 (Pin_1), ACN2.2 (Pin_2), C32.2, R25.1
- net at U4.2 ((PCINT3/XTAL1/CLKI/OC1B*/ADC3)_PB3): now also C13.2, R10.2
- net at U4.5 (PB0_(MOSI/DI/SDA/AIN0/OC0A/OC1A/AREF/PCINT0)): now also R21.1, R23.1
- net at LED1.2 (A): now also R21.2; no longer R22.1
- net at C4.1, C7.1, R5.1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: now also D1.1 (+)
- net at LF1.3: now also D1.2
- net at LF1.4: now also D1.3
- new net: C31.1, R24.2, R25.2
- new net: T1.3 (SA), U2.2
- new net: R24.1, U5.6
- new net: LED2.2 (A), R22.1
- new net: G1.1 (Pin_1), G1.2 (Pin_2), R26.1, U5.4
- new net: R23.2, U5.1
- no-connect marks 0 -> 10
Other:
- moved on the sheet: A2, ACL1, ACN1, C1, C12, C14, C15, C16, C17, C18, C19, C2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
