File: kicad/ELSONIC/POWER_BD_SV2/POWER_BD_SV2.kicad_sch (KiCad schematic)
At the start: 97 parts, among them J2 SMW250-06P, J3 SMW250-02P, T1 EI2811BP, T2 EER28, U1 ICE3BR0665J, U2 H11AA1, U3 PC817, U4 ATTINY85-20PU_1, U5 MOC3021M, U6 LM7805_TO220

Commit message: 자동보정 구현: minDim/maxDim 기준 - setup()에서 ZC 주기 측정 후 minDim/maxDim 동적 계산 - maxDim = avgPeriod - 6 (margin) - minDim = avgPeriod * 62 / 166 - 2 - 50Hz/60Hz 및 오실레이터 편차 자동 대응
Parts:
- C11, C13: footprint 04_MyFoot_Passive:C_Disc_D6.0mm_P5.00mm -> 04_MyFoot_Passive:C_3216Metric
- C12, C26, C27, C28, C30, C5, C9: footprint 04_MyFoot_Passive:C_Disc_D4.7mm_T3.0mm_P5.00mm -> 04_MyFoot_Passive:C_3216Metric
- C15, C19, C6, C8: footprint 04_MyFoot_Passive:C_Disc_D4.7mm_P5.00mm -> 04_MyFoot_Passive:C_3216Metric
- LED1, LED2: footprint 03_MyFoot_Active:LED_D3.0mm -> 03_MyFoot_Active:LED_2012Metric
- R10, R11, R12, R13, R14, R15, R16, R17, R2, R20, R21, R22, R23, R6, R7, R8, R9: footprint 04_MyFoot_Passive:R_Axial_0.25W_P10.16mm -> 04_MyFoot_Passive:R_3216Metric
Changed lines of the file:
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@@
 			)
 		)
-		(property "Footprint" "04_MyFoot_Passive:R_Axial_0.25W_P10.16mm"
+		(property "Footprint" "04_MyFoot_Passive:R_3216Metric"
 			(at 110.744 172.466 90)
 			(effects
@@
 			)
 		)
-		(property "Footprint" "04_MyFoot_Passive:R_Axial_0.25W_P10.16mm"
+		(property "Footprint" "04_MyFoot_Passive:R_3216Metric"
 			(at 126.746 87.884 90)
 			(effects
@@
 			)
 		)
-		(property "Footprint" "04_MyFoot_Passive:R_Axial_0.25W_P10.16mm"
+		(property "Footprint" "04_MyFoot_Passive:R_3216Metric"
 			(at 272.796 195.834 90)
 			(effects
@@
 			)
 		)
-		(property "Footprint" "04_MyFoot_Passive:R_Axial_0.25W_P10.16mm"
+		(property "Footprint" "04_MyFoot_Passive:R_3216Metric"
 			(at 132.334 92.964 90)
 			(effects
@@
 			)
 		)
-		(property "Footprint" "04_MyFoot_Passive:C_Disc_D4.7mm_P5.00mm"
+		(property "Footprint" "04_MyFoot_Passive:C_3216Metric"
 			(at 232.41 132.3848 0)
 			(effects
@@
 			)
 		)
-		(property "Footprint" "04_MyFoot_Passive:R_Axial_0.25W_P10.16mm"
+		(property "Footprint" "04_MyFoot_Passive:R_3216Metric"
 			(at 147.574 171.196 90)
 			(effects
@@
 			)
 		)
-		(property "Footprint" "04_MyFoot_Passive:R_Axial_0.25W_P10.16mm"
+		(property "Footprint" "04_MyFoot_Passive:R_3216Metric"
 			(at 65.024 175.514 90)
 			(effects
@@
 			)
 		)
-		(property "Footprint" "04_MyFoot_Passive:C_Disc_D4.7mm_P5.00mm"
+		(property "Footprint" "04_MyFoot_Passive:C_3216Metric"
 			(at 215.9 123.4948 0)
 			(effects
@@
 			)
 		)
-		(property "Footprint" "04_MyFoot_Passive:C_Disc_D4.7mm_T3.0mm_P5.00mm"
+		(property "Footprint" "04_MyFoot_Passive:C_3216Metric"
 			(at 147.6248 181.61 0)
 			(effects
@@
 			)
 		)
-		(property "Footprint" "04_MyFoot_Passive:C_Disc_D4.7mm_T3.0mm_P5.00mm"
+		(property "Footprint" "04_MyFoot_Passive:C_3216Metric"
 			(at 95.25 110.7948 0)
 			(effects
@@
 			)
 		)
-		(property "Footprint" "04_MyFoot_Passive:R_Axial_0.25W_P10.16mm"
+		(property "Footprint" "04_MyFoot_Passive:R_3216Metric"
 			(at 147.574 213.614 90)
 			(effects
@@
 			)
 		)
-		(property "Footprint" "03_MyFoot_Active:LED_D3.0mm"
+		(property "Footprint" "03_MyFoot_Active:LED_2012Metric"
 			(at 274.32 105.41 0)
 			(effects
@@
 			)
 		)
-		(property "Datasheet" "~"
+		(property "Datasheet" ""
 			(at 274.32 105.41 0)
 			(effects
@@
 			)
 		)
-		(property "Description" "Light emitting diode"
+		(property "Description" ""
 			(at 274.32 105.41 0)
 			(effects
@@
 			)
 		)
-		(property "Sim.Pins" "1=K 2=A"
+		(property "Sim.Pins" ""
 			(at 274.32 105.41 0)
 			(effects
@@
 			)
 		)
-		(property "Footprint" "04_MyFoot_Passive:C_Disc_D4.7mm_T3.0mm_P5.00mm"
+		(property "Footprint" "04_MyFoot_Passive:C_3216Metric"
 			(at 261.9248 92.71 0)
 			(effects
@@
 			)
 		)
-		(property "Footprint" "04_MyFoot_Passive:R_Axial_0.25W_P10.16mm"
+		(property "Footprint" "04_MyFoot_Passive:R_3216Metric"
 			(at 273.304 93.726 90)
 			(effects
@@
 			)
 		)
-		(property "Footprint" "04_MyFoot_Passive:R_Axial_0.25W_P10.16mm"
+		(property "Footprint" "04_MyFoot_Passive:R_3216Metric"
 			(at 205.994 25.654 90)
 			(effects
@@
 			)
 		)
-		(property "Footprint" "04_MyFoot_Passive:C_Disc_D4.7mm_P5.00mm"
+		(property "Footprint" "04_MyFoot_Passive:C_3216Metric"
 			(at 110.7948 113.03 0)
 			(effects
@@
 			)
 		)
-		(property "Footprint" "04_MyFoot_Passive:C_Disc_D4.7mm_P5.00mm"
+		(property "Footprint" "04_MyFoot_Passive:C_3216Metric"
 			(at 117.1448 184.15 0)
 			(effects
@@
 			)
 		)
-		(property "Footprint" "04_MyFoot_Passive:R_Axial_0.25W_P10.16mm"
+		(property "Footprint" "04_MyFoot_Passive:R_3216Metric"
 			(at 136.144 206.756 90)
 			(effects
@@
 			)
 		)
-		(property "Footprint" "04_MyFoot_Passive:C_Disc_D6.0mm_P5.00mm"
+		(property "Footprint" "04_MyFoot_Passive:C_3216Metric"
 			(at 136.1948 218.44 0)
 			(effects
@@
 			)
 		)
-		(property "Footprint" "04_MyFoot_Passive:C_Disc_D4.7mm_T3.0mm_P5.00mm"
+		(property "Footprint" "04_MyFoot_Passive:C_3216Metric"
 			(at 124.7648 113.03 0)
 			(effects
@@
 			)
 		)
-		(property "Footprint" "04_MyFoot_Passive:R_Axial_0.25W_P10.16mm"
+		(property "Footprint" "04_MyFoot_Passive:R_3216Metric"
 			(at 278.384 185.674 90)
 			(effects
@@
 			)
 		)
-		(property "Footprint" "04_MyFoot_Passive:R_Axial_0.25W_P10.16mm"
+		(property "Footprint" "04_MyFoot_Passive:R_3216Metric"
 			(at 183.134 132.334 90)
 			(effects
@@
 			)
 		)
-		(property "Footprint" "04_MyFoot_Passive:R_Axial_0.25W_P10.16mm"
+		(property "Footprint" "04_MyFoot_Passive:R_3216Metric"
 			(at 212.344 132.334 90)
 			(effects
@@
 			)
 		)
-		(property "Footprint" "03_MyFoot_Active:LED_D3.0mm"
+		(property "Footprint" "03_MyFoot_Active:LED_2012Metric"
 			(at 271.78 205.74 0)
 			(effects
@@
 			)
 		)
-		(property "Footprint" "04_MyFoot_Passive:C_Disc_D6.0mm_P5.00mm"
+		(property "Footprint" "04_MyFoot_Passive:C_3216Metric"
 			(at 155.2448 218.44 0)
 			(effects
@@
 			)
 		)
-		(property "Footprint" "04_MyFoot_Passive:R_Axial_0.25W_P10.16mm"
+		(property "Footprint" "04_MyFoot_Passive:R_3216Metric"
 			(at 239.014 148.336 90)
 			(effects
@@
 			)
 		)
-		(property "Footprint" "04_MyFoot_Passive:R_Axial_0.25W_P10.16mm"
+		(property "Footprint" "04_MyFoot_Passive:R_3216Metric"
 			(at 205.994 87.884 90)
 			(effects
@@
 			)
 		)
-		(property "Footprint" "04_MyFoot_Passive:R_Axial_0.25W_P10.16mm"
+		(property "Footprint" "04_MyFoot_Passive:R_3216Metric"
 			(at 205.994 61.214 90)
 			(effects
@@
 			)
 		)
-		(property "Footprint" "04_MyFoot_Passive:C_Disc_D4.7mm_T3.0mm_P5.00mm"
+		(property "Footprint" "04_MyFoot_Passive:C_3216Metric"
 			(at 319.0748 91.44 0)
 			(effects
@@
 			)
 		)
-		(property "Footprint" "04_MyFoot_Passive:R_Axial_0.25W_P10.16mm"
+		(property "Footprint" "04_MyFoot_Passive:R_3216Metric"
 			(at 195.834 124.206 90)
 			(effects
@@
 			)
 		)
-		(property "Footprint" "04_MyFoot_Passive:C_Disc_D4.7mm_T3.0mm_P5.00mm"
+		(property "Footprint" "04_MyFoot_Passive:C_3216Metric"
 			(at 261.9248 30.48 0)
 			(effects
@@
 			)
 		)
-		(property "Footprint" "04_MyFoot_Passive:C_Disc_D4.7mm_T3.0mm_P5.00mm"
+		(property "Footprint" "04_MyFoot_Passive:C_3216Metric"
 			(at 261.9248 66.04 0)
 			(effects

Commit message: 프로젝트 전체 정리: KiCAD 파일 업데이트, 불필요한 파일 삭제
Parts:
- C11: value MLCC475 -> NOT
- L1: value 2.2uH/4.2A -> 22uH/4.2A
- L2: value 2.2uH/4.2A -> 10uH/4.2A
- L3: value 2.2uH/4.2A -> 4.7uH/4.2A
- R10: value 3.3K -> 4.7K
- R18: value 20K -> 1K
- R19: value 18K -> 40K
- R2: value 1K -> 1.2K
- R21: value 1K -> 3.3K
- R22: value 680R -> 4.7K
- R23: value 330R -> 220R
- R9: value 4.7K -> 1K
