File: kicad/ELSONIC/POWER_BD_SV3/POWER_BD_SV3.kicad_pcb (KiCad board)
At the start: 2 copper layers, 150 x 98 mm, 97 parts, among them J2 SMW250-06P, J3 SMW250-02P, T1 EI2811BP, T2 EER28, U1 ICE3BR0665J, U2 H11AA1, U3 PC817, U4 ATTINY85-20PU_1, U5 MOC3021M, U6 LM7805_TO220

Commit message: JLCPCB에 POWER_BD주문
Parts:
- added R27: 100R, 04_MyFoot_Passive:R_3216Metric, F.Cu at (89.5, -8.50)
- added RV2: 3362P103, 04_MyFoot_Passive:TRIM_3362P, F.Cu at (82.5, -4.29)
- C11, C13: value MLCC475 -> MLCC335; footprint 04_MyFoot_Passive:C_Disc_D6.0mm_P5.00mm -> 04_MyFoot_Passive:C_3216Metric
- C12, C26, C27, C28, C30, C5, C9: footprint 04_MyFoot_Passive:C_Disc_D4.7mm_T3.0mm_P5.00mm -> 04_MyFoot_Passive:C_3216Metric
- C15, C19, C6, C8: footprint 04_MyFoot_Passive:C_Disc_D4.7mm_P5.00mm -> 04_MyFoot_Passive:C_3216Metric
- C31: footprint 04_MyFoot_Passive:C_PP_L23.0mm_W10.9mm_P21.2mm -> 04_MyFoot_Passive:C_PP_P10.0mm_P21.2mm
- C7: value CC472/630V -> CC472/1kV
- D3: value UF4004 -> UF4007
- L1, L2, L3: value 2.2uH/4.2A -> 10uH/4.2A
- LED1, LED2: value RED/3Pi -> LED_SMD; footprint 03_MyFoot_Active:LED_D3.0mm -> 03_MyFoot_Active:LED_2012Metric
- R10: value 3.3K -> 4.7K; footprint 04_MyFoot_Passive:R_Axial_0.25W_P10.16mm -> 04_MyFoot_Passive:R_3216Metric
- R11, R12, R14, R15, R16, R17, R6, R7, R8: footprint 04_MyFoot_Passive:R_Axial_0.25W_P10.16mm -> 04_MyFoot_Passive:R_3216Metric
- R13: value 1.2K -> 1.2K/F; footprint 04_MyFoot_Passive:R_Axial_0.25W_P10.16mm -> 04_MyFoot_Passive:R_3216Metric
- R18: value 20K -> 1K/F; footprint 04_MyFoot_Passive:R_Axial_0.25W_P10.16mm -> 04_MyFoot_Passive:R_3216Metric
- R19: value 18K -> 40K/F; footprint 04_MyFoot_Passive:R_Axial_0.25W_P10.16mm -> 04_MyFoot_Passive:R_3216Metric
- R2, R21: value 1K -> 1.2K; footprint 04_MyFoot_Passive:R_Axial_0.25W_P10.16mm -> 04_MyFoot_Passive:R_3216Metric
- R20: value 10K -> 10K/F; footprint 04_MyFoot_Passive:R_Axial_0.25W_P10.16mm -> 04_MyFoot_Passive:R_3216Metric
- R22: value 680R -> 2.2K; footprint 04_MyFoot_Passive:R_Axial_0.25W_P10.16mm -> 04_MyFoot_Passive:R_3216Metric
- R23: value 330R -> 220R; footprint 04_MyFoot_Passive:R_Axial_0.25W_P10.16mm -> 04_MyFoot_Passive:R_3216Metric
- R9: value 4.7K -> 1K; footprint 04_MyFoot_Passive:R_Axial_0.25W_P10.16mm -> 04_MyFoot_Passive:R_3216Metric
- moved LED2 68.7 mm to (7.20, -52.0), turned to 0 degrees
- moved R22 66.2 mm to (7.00, -57.0)
- moved R2 25.1 mm to (118.0, -22.5)
- moved C13 20.6 mm to (63.5, -12.0), turned to 0 degrees
- moved C15 20.1 mm to (63.5, -24.0), turned to 0 degrees
- moved R6 19.6 mm to (109.0, -21.0)
- moved LED1 19.6 mm to (92.0, -3.50), turned to 0 degrees
- moved C11 17.2 mm to (63.5, -15.0), turned to 0 degrees
- moved C12 14.0 mm to (85.5, -19.0), turned to 180 degrees
- moved C19 12.8 mm to (63.5, -18.0), turned to 180 degrees
- moved R20 11.0 mm to (55.5, -18.0), turned to 0 degrees
- moved VR1 10.4 mm to (55.5, -25.0)
- moved C9 10.2 mm to (54.5, -33.6), turned to 180 degrees
- moved U2 8.12 mm to (128.5, -13.0)
- moved C8 7.73 mm to (118.0, -19.0), turned to 180 degrees
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Connections:
- C11 pad 2: /PWM_PW -> Net-(U4-(PCINT3/XTAL1/CLKI/OC1B*/ADC3)_PB3)
- R21 pad 1: Net-(U4-PB0_(MOSI/DI/SDA/AIN0/OC0A/OC1A/AREF/PCINT0)) -> Net-(U4-PB1_(MISO/DO/AIN1/OC0B/OC1A*/PCINT1))
- R22 pad 2: +8V -> +24V
- U4 pad 3: unconnected-(U4-(PCINT4/XTAL2/CLKO/OC1B/ADC2)_PB4-Pad3) -> Net-(U4-(PCINT4/XTAL2/CLKO/OC1B/ADC2)_PB4)
- U4 pad 6: unconnected-(U4-PB1_(MISO/DO/AIN1/OC0B/OC1A*/PCINT1)-Pad6) -> Net-(U4-PB1_(MISO/DO/AIN1/OC0B/OC1A*/PCINT1))
Routing:
- net GND: track 0.00 -> 52.8 mm, vias 0 -> 2
- net Net-(T1-SB): track 28.5 -> 7.01 mm
- net Net-(C15-Pad1): track 53.2 -> 32.9 mm, vias 0 -> 1
- net Net-(U4-(PCINT3/XTAL1/CLKI/OC1B*/ADC3)_PB3): track 17.2 -> 36.2 mm, vias 0 -> 1
- net +5V: track 187.4 -> 168.5 mm, vias 0 -> 2
- net Net-(C15-Pad2): track 20.7 -> 6.00 mm
- net Earth: track 192.9 -> 207.3 mm
- net +12V: track 107.8 -> 94.4 mm
- net Net-(U4-(PCINT5/RESET*/ADC0/dW)_PB5): track 33.2 -> 20.8 mm, vias 0 -> 1
- net Net-(C31-Pad1): track 41.4 -> 53.5 mm
- net Net-(U4-PB1_(MISO/DO/AIN1/OC0B/OC1A*/PCINT1)): track 0.00 -> 10.2 mm
- net Net-(T2-N2): track 45.2 -> 54.6 mm
- net /ZVC: track 44.2 -> 35.8 mm
- net Net-(C18-Pad1): track 12.0 -> 4.35 mm
- net Net-(R27-Pad1): track 0.00 -> 7.04 mm
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- added copper zone on B.Cu, net /N01
Other:
- outline, holes or cut-outs redrawn
- board text added: "POWER_BD_SV2.0"
- board text removed: "POWER_BD_NV2.0"
