File: kicad/ELSONIC/POWER_BD_SV3/POWER_BD_SV3.kicad_sch (KiCad schematic)
At the start: 99 parts, among them J2 SMW250-06P, J3 SMW250-02P, T1 EI2811BP, T2 EER28, U1 ICE3BR0665J, U2 H11AA1, U3 PC817, U4 ATTINY85-20PU_1, U5 MOC3021M, U6 LM7805_TO220

Commit message: feat: update ultrasonic controller and board design
Other:
- note added: "220VAC_L"
- note added: "220VAC_N"
Changed lines of the file:
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@@
 	(generator_version "10.0")
 	(paper "A3")
+	(text "220VAC_L"
+		(exclude_from_sim no)
+		(at 35.814 254.762 0)
+		(effects
+			(font
+				(size 1.397 1.397)
+			)
+		)
+	)
+	(text "220VAC_N"
+		(exclude_from_sim no)
+		(at 35.56 244.602 0)
+		(effects
+			(font
+				(size 1.397 1.397)
+			)
+		)
+	)
 	(junction
 		(at 256.54 76.2)
