File: kicad/ELSONIC/KI_Mega_PWBD/KI_Mega_PWBD.kicad_sch (KiCad schematic)
At the start: 10 parts, among them J1 SMW250-02P, J4 SMW250-03P

Commit message: ms_board_V3 회로설계 1차 내용정리
Parts:
- added C1, C2, C3: C, symbol Device:C
- added C1-2: 1uK63, symbol 04_MyLib_Passive:C
- added C10, C6, C7: 0.1uF/630V, symbol 04_MyLib_Passive:C
- added C107: MLCC330, symbol 04_MyLib_Passive:C
- added C11: CR1201, symbol 04_MyLib_Passive:CR1201
- added C12, C13, C4, C5, C8, C9, MC1: C, symbol 04_MyLib_Passive:C
- added C14, C15: 10pF, symbol 04_MyLib_Passive:C
- added C16, C17: 10nF, symbol 04_MyLib_Passive:C
- added CT2: CTL-6-P, symbol 04_MyLib_Passive:CTL-6_P
- added D1, D1-2, D10, D5: UF4007, Diode_THT:D_DO-41_SOD81_P10.16mm_Horizontal, symbol 03_MyLib_Active:UF4007
- added D2, D3, D4, D6, D9: 1N47xxA, Diode_THT:D_DO-41_SOD81_P10.16mm_Horizontal, symbol Diode:1N47xxA
- added D2-1, D2-2, D2-3: 1N4148, Diode_THT:D_DO-35_SOD27_P7.62mm_Horizontal, symbol 03_MyLib_Active:1N4148
- added D7: FMU34S, symbol 03_MyLib_Active:FMU34S
- added D8: FMG34R, symbol 03_MyLib_Active:FMG34R
- added FC1: 470uF/25V, symbol 04_MyLib_Passive:C_Pol
- added FC2: 220uF/25V, symbol 04_MyLib_Passive:C_Pol
- added FC3, FC4, FC5: 100uF/400V, symbol 04_MyLib_Passive:C_Pol
- added FC6: 10uF/50V, symbol 04_MyLib_Passive:C_Pol
- added J1, J1-2, J116: SMW250-02P, SMW25002, symbol 02_MyLib_Connectors:SMW250-02P
- added J2: SMW250-03P, SHDR11W64P0X250_1X03, symbol 02_MyLib_Connectors:SMW250-03P
- added J2-2: SMW250-05P, symbol 02_MyLib_Connectors:SMW250-05P
- added J5: SMW250-04P, SHDR11W64P0X250_1X04, symbol 02_MyLib_Connectors:SMW250-04P
- added K2-1, K2-2, K2-3: G6A, Relay_THT:Relay_DPDT_Omron_G6A, symbol 05_MyLib_Others:G6A
- added L1, L2-1, L2-2, L2-3, L2-4, L4: Inductor, symbol 04_MyLib_Passive:Inductor
- added PZT1, PZT2: Transducer, symbol Device:Crystal
- added Q1, Q2, Q3, Q4: 2SK2932, symbol 03_MyLib_Active:2SK2932
- added Q5: KTC3198-Y, TO92250P470H770-3, symbol 03_MyLib_Active:KTC3198-Y
- added R1, R2, R3, R4, R5: R, symbol 04_MyLib_Passive:R
- added R1-2, R2-2: 15K, symbol 04_MyLib_Passive:R
- added R10, R6: 5.1R/1W, symbol 04_MyLib_Passive:R
- added R107: 330K/1W, symbol 04_MyLib_Passive:R
- added R108: 820K, symbol 04_MyLib_Passive:R
- added R11, R7: 0.68R/1W, symbol 04_MyLib_Passive:R
- added R12, R13, R14: 15K/5W, symbol 04_MyLib_Passive:R
- added R15: 10K, symbol 04_MyLib_Passive:R
- added R16: 4.7K, symbol 04_MyLib_Passive:R
- added R17, R19, R25, R26: 50R, symbol 04_MyLib_Passive:R
- added R18, R20, R8, R9: 270R, symbol 04_MyLib_Passive:R
- added R21, R22, R23, R24: 25R, symbol 04_MyLib_Passive:R
- added R3-2: 1.5K, symbol 04_MyLib_Passive:R
- added R30, R32: NC, symbol Device:R
- added R31: 10R, symbol Device:R
- added R4-2: 220K, symbol 04_MyLib_Passive:R
- added RV1-2: RJ6S203, symbol 04_MyLib_Passive:R_POT
- added SCR1, SCR2: SG10GZ47, symbol 03_MyLib_Active:SG10GZ47
- added T1: Transformer_1P_1S, symbol 04_MyLib_Passive:Transformer_1P_1S
- added T2: OUTPUT_TRANS, symbol 04_MyLib_Passive:Transformer_1P_1S
- added TR1: PULSE_TR_RING, symbol 04_MyLib_Passive:PULSE_TR_RING
- added U1: HD29026A, Package_DIP:DIP-8_W7.62mm, symbol 01_MyLib_ICs:HD29026A
- added U10, U9: LTC5507ES6, Package_TO_SOT_SMD:TSOT-23-6, symbol RF:LTC5507ES6
- added U2: LM7812_TO220, Package_TO_SOT_THT:TO-220-3_Vertical, symbol Regulator_Linear:LM7812_TO220
- added U2-1: ULN2003, symbol 01_MyLib_ICs:ULN2003
- added U3: 74HC04, symbol 74xx:74HC04
- added U4: 74HC390N, symbol 01_MyLib_ICs:74HC390N
- added U5: PC817X3NSZ1B, DIP762W50P254L495H455Q4, symbol 01_MyLib_ICs:PC817X3NSZ1B
- added U6: 74HC14, symbol 74xx:74HC14
- added U7: AMS1117-3.3, Package_TO_SOT_SMD:SOT-223-3_TabPin2, symbol Regulator_Linear:AMS1117-3.3
- added U8: LM2576S-5, Package_TO_SOT_SMD:TO-263-5_TabPin3, symbol Regulator_Switching:LM2576S-5
- C1-1: renamed from C1; value C -> 1uK63
- R1-1: renamed from R1; value R -> 22K
- R2-1: renamed from R2; value R -> 15K
- R3-1: renamed from R3; value R -> 10K
- R4-1: renamed from R4; value R -> 120K
- RV1-1: renamed from RV1; value R_POT -> RJ6S203
- renumbered D1 to D1-1, J1 to J1-1
Connections:
- net at C1-1.1, J1-1.2, J4.1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: now also CT1.2, C1-2.1, J1-2.2, PZT1.1, R2-2.1, R4-2.1, RV1-2.1, T1.4 (SB); no longer CT1.1
- net at CT1.3, J4.3, R1-1.2: now also PZT1.2, R1-2.2, R30.2
- net at CT1.4: now also L4.2
- new net: K2-1.11, K2-1.21, K2-2.12, K2-2.22, L2-1.2, L2-2.1
- new net: K2-2.11, K2-2.21, K2-3.12, K2-3.22, L2-2.2, L2-3.1
- new net: D2-2.2 (A), K2-2.A2, U2-1.15 (O2)
- new net: J5.3, R30.1
- new net: K2-3.11, K2-3.21, L2-3.2, T1.3 (SA)
- new net: D10.1 (K), FC6.1, R15.2
- new net: D10.2 (A), R107.2
- new net: J116.1, R5.2, U1.2 (1A), U3.1
- new net: J116.2, U1.4 (2A), U3.2
- new net: C6.2, C7.1, FC3.2, FC4.1, R12.1, R13.2, T1.2 (AB)
- new net: D2-3.2 (A), K2-3.A2, U2-1.14 (O3)
- new net: C2.1, R1.1, U1.7 (OUT_1Y)
- new net: C2.2, Q1.1 (G), R1.2, R2.1
- new net: C107.1, D9.1 (K), Q5.3, R108.2
- new net: D4.1 (K), Q3.2 (D), R11.1, T1.1 (AA), TR1.7
- new net: Q4.3 (S), R11.2
- new net: D4.2 (A), D6.2 (A)
- new net: R18.1, R20.1, TR1.6
- new net: C4.1, D1.1 (K), R18.2
- new net: C14.2, CT2.1, R17.2, R21.2, R22.2
- new net: C15.2, CT2.2, R19.2, R23.2, R24.2
- new net: C14.1, CT2.3, L2-4.1
- new net: C15.1, CT2.4, PZT2.2
- new net: R5.1, U4.3 (1Q0)
- new net: J5.1, J5.4, R32.1
- new net: J5.2, R31.1, R32.2
- new net: C4.2, D1.2 (A), D3.1 (K), R20.2, R6.1
- new net: J2-2.1, U2-1.1 (I1)
- new net: D2-1.2 (A), K2-1.A2, U2-1.16 (O1)
- new net: J2-2.2, U2-1.2 (I2)
- new net: J2-2.3, U2-1.3 (I3)
- new net: C11.1, D7.1 (A), D8.3 (K), SCR1.2 (A), SCR2.1 (K)
- new net: C5.2, D5.2 (A), D6.1 (K), R10.1, R9.2
- new net: C1-2.2, D1-2.1 (K), J1-2.1, R4-2.2
- new net: C17.1, U9.6 (RF_{IN})
- new net: R8.1, R9.1, TR1.8
- new net: C5.1, D5.1 (K), R8.2
- new net: D7.2 (K), FC5.1, L1.1
- new net: C3.2, Q2.1 (G), R3.2, R4.1
- new net: C16.2, U10.6 (RF_{IN})
- new net: Q3.1 (G), R6.2
- new net: Q3.3 (S), R7.2
- new net: C107.2, R15.1, U5.1
- new net: Q1.2 (D), TR1.1
- new net: D2.2 (A), D3.2 (A)
- new net: CT1.1, R31.2
- new net: C3.1, R3.1, U1.5 (OUT_2Y)
- new net: R3-2.1, RV1-2.3
- new net: R1-2.1, R2-2.2, R3-2.2
- new net: D1-2.2 (A), RV1-2.2
- new net: Q5.2, U5.2
- new net: Q4.1 (G), R10.2
- new net: K2-1.12, K2-1.22, L2-1.1, L4.1
- new net: L2-4.2, T2.4 (SB)
- new net: Q2.2 (D), TR1.4
- new net +12V: C12.1, C13.1, FC2.1, MC1.1, U1.6 (Vcc), U2.3 (VO)
- new net +15V: C8.1, C9.1, FC1.1, J1.2, TR1.2, TR1.3, U2.1 (VI)
- new net +5V: C1.1, D2-1.1 (K), D2-2.1 (K), D2-3.1 (K), J2-2.5, K2-1.A1, K2-2.A1, K2-3.A1, R16.2, U2-1.9 (COM)
- new net AC220L: C11.2, J2.1, R107.1, R108.1, SCR1.1 (K), SCR2.2 (A)
- new net AC220N: D7.3 (A), D8.1 (K), D9.2 (A), FC6.2, J2.3, Q5.1
- new net FWD: C17.2, R21.1, R22.1, R25.2
- new net GND: C1.2, C12.2, C13.2, C8.2, C9.2, FC1.2, FC2.2, J1.1, J2-2.4, MC1.2, PZT2.1, Q1.3 (S), Q2.3 (S), R17.1, R19.1, R2.2, R25.1, R26.1, R4.2, T2.3 (SA), U1.3 (GND), U2-1.8 (GND), U2.2 (GND), U3.3, U5.3
- new net PA0: U9.3 (V_{OUT})
- new net PA1: U10.3 (V_{OUT})
- new net REV: C16.1, R23.1, R24.1, R26.2
- new net VPP: C10.2, C7.2, FC3.1, L1.2, Q4.2 (D), R12.2, R14.2
- new net VSS: C10.1, C6.1, D2.1 (K), D8.2 (A), FC4.2, FC5.2, R13.1, R14.1, R7.1, TR1.5
- new net ZERO_CROSS: R16.1, U5.4
Other:
- moved on the sheet: C1-1, CT1, D1-1, J1-1, J4, R1-1, R2-1, R3-1, R4-1, RV1-1
