File: kicad/ELSONIC/Multi_Mega_Main_V2/Multi_Mega_Main_V2.kicad_sch (KiCad schematic)
At the start: 186 parts, among them IC1 LM5005MHX_NOPB, J1 SMW250-02P, J2 Conn_01x04, J3 Conn_ARM_SWD_10, J4 Conn_01x02, J5 Conn_01x03, J6 Conn_01x06, J7 SMW250-02P, J8 Conn_02x13_Top_Bottom, J9 Conn_02x10_Odd_Even, K1 G6A274, K2 PA1A_5V, K3 PA1A_5V, K4 G6A274, K5 PA1A_5V, K6 G6A274, K7 PA1A_5V, K8 PA1A_5V, K9 G6A274, Q1 STD25N10F7, Q2 STD25N10F7, SW1 SW_Push, SW2 SW_DIP_x02, T1 OUTPUT_Transformer, U1 AMS1117-3.3, U10 TLP185, U11 TLP185, U12 TLP185, U2 UCC21520DW, U3 STM32G474RBT6, U4 INA190A4, U5 MAX3485, U6 TLP185, U7 ULN2003, U8 ULN2003, U9 TLP185, Y1 HC-49SMD

Commit message: chore: KiCad 아트웍 및 라이브러리 변경 반영
Parts:
- removed C17: CL104K, 04_MyFoot_Passive:C_2012Metric, symbol 04_MyLib_Passive:C_Small
- removed CT1: CT_TR, symbol 04_MyLib_Passive:CT_TROID
- removed D1: BAV99, Package_TO_SOT_SMD:SOT-23, symbol Diode:BAV99
- removed D2, D3: SS24, Diode_SMD:D_SMA, symbol Diode:SS24
- removed DCDC1, DCDC2: MUS2415N, Converter_DCDC:Converter_DCDC_TRACO_TME_24xxS_Single_THT, symbol Converter_DCDC:TME-2415S
- removed J2: Conn_01x04, symbol Connector_Generic:Conn_01x04
- removed J3: Conn_ARM_SWD_10, symbol 02_MyLib_Connectors:Conn_ARM_SWD_10
- removed J4: Conn_01x02, symbol Connector_Generic:Conn_01x02
- removed J5: Conn_01x03, symbol Connector_Generic:Conn_01x03
- removed J6: Conn_01x06, symbol Connector_Generic:Conn_01x06
- removed J8: Conn_02x13_Top_Bottom, symbol Connector_Generic:Conn_02x13_Top_Bottom
- removed J9: Conn_02x10_Odd_Even, symbol Connector_Generic:Conn_02x10_Odd_Even
- removed Q1, Q2: STD25N10F7, Package_TO_SOT_SMD:TO-252-2, symbol Transistor_FET:STD7NK40Z
- removed T1: OUTPUT_Transformer, symbol 04_MyLib_Passive:Transformer_1P_1S
- removed U4: INA190A4, Package_TO_SOT_SMD:SOT-363_SC-70-6, symbol 01_MyLib_ICs:INA190A4
- removed U5: MAX3485, Package_SO:SOIC-8_3.9x4.9mm_P1.27mm, symbol Interface_UART:MAX3485
- removed U7, U8: ULN2003, symbol 01_MyLib_ICs:ULN2003
- removed Y1: HC-49SMD, 03_MyFoot_Active:Crystal_SMD_HC49-SD, symbol 03_MyLib_Active:Crystal
- added D1: BAV99, 03_MyFoot_Active:SOT-23, symbol 03_MyLib_Active:BAV99
- added D17, D18: MM3Z3V6, 03_MyFoot_Active:D_SOD-323_HandSoldering, symbol 03_MyLib_Active:MM3Z3V6
- added D2, D3: SS24B, 03_MyFoot_Active:D_SMB, symbol 03_MyLib_Active:SS24B
- added DCDC1, DCDC2: MUS2415N, 05_MyFoot_Others:MUS2415N, symbol 05_MyLib_Others:MUS2415N
- added H1, H2: MountingHole_Pad, 06_MyFoot_Mechanical:MTHole_3.5mm_6.8mmPad_GND, symbol 06_MyLib_Mechanical:MountingHole_Pad
- added H3, H4: MountingHole, 06_MyFoot_Mechanical:MTHole_3.5mm, symbol 06_MyLib_Mechanical:MountingHole
- added J2: Screw_Terminal_01x06, 02_MyFoot_Connectors:TB_P5.00mm_6P, symbol 06_MyLib_Mechanical:Screw_Terminal_01x06
- added J3: ARM_SWD_10, 02_MyFoot_Connectors:IDC-Header_2x05_P2.54mm_Vertical, symbol 02_MyLib_Connectors:Conn_02x05_Odd_Even
- added J4: Conn_01x06_HEADERPIN, 02_MyFoot_Connectors:PinHeader_1x06_P2.54mm_Vertical, symbol 02_MyLib_Connectors:Conn_01x06_HEADERPIN
- added J5: Conn_01x03, 02_MyFoot_Connectors:PinHeader_1x03_P2.54mm_Vertical, symbol 02_MyLib_Connectors:Conn_01x03
- added J6: Conn_02x10_Odd_Even, 02_MyFoot_Connectors:IDC-Header_2x10_P2.54mm_Vertical, symbol 02_MyLib_Connectors:Conn_02x10_Odd_Even
- added J8: Conn_02x13_Odd_Even, 02_MyFoot_Connectors:IDC-Header_2x13_P2.54mm_Latch_Vertical, symbol 02_MyLib_Connectors:Conn_02x13_Odd_Even
- added Q1, Q2: STD25N10F7, Package_TO_SOT_SMD:TO-252-2, symbol 03_MyLib_Active:STD7N10F7
- added R49, R50: W4J0102, 04_MyFoot_Passive:R_3216Metric, symbol 04_MyLib_Passive:R
- added R51: W4F0000, 04_MyFoot_Passive:R_3216Metric, symbol 04_MyLib_Passive:R
- added T1: TOROID_OUTPUT_OD20_T6T12, 04_MyFoot_Passive:Toroid_OD20mm_ID10-T6T12, symbol 04_MyLib_Passive:TOROID_OUTPUT_OD20_T6T12
- added T2: TOROID_CT_OD16_T1T20, 04_MyFoot_Passive:Toroid_OD16mm_ID9.6-T1T20, symbol 04_MyLib_Passive:TOROID_CT_OD16_T1T20
- added U4: INA190A3IDCKR, Package_TO_SOT_SMD:SOT-363_SC-70-6, symbol 01_MyLib_ICs:INA190A3
- added U5: MAX3485ESA, 01_MyFoot_ICs:SOIC-8_3.9x4.9mm_P1.27mm, symbol 01_MyLib_ICs:MAX3485ESA
- added U7, U8: ULN2003ADR, 01_MyFoot_ICs:SOIC-16_3.9x9.9mm_P1.27mm, symbol 01_MyLib_ICs:ULN2003ADR
- added Y1: X49SM8M, 03_MyFoot_Active:Crystal_SMD_HC49-SD, symbol 03_MyLib_Active:X49SM8M
- C1, C11, C13, C14, C15, C16, C19, C21, C23, C28, C30, C33, C4, C5, C52, C53, C60, C62, C64, C66, C7, C9: value CL104K -> CL21B104K; LCSC (none) -> C1711
- C10, C31: value 10UF25V -> 10UF25V67RV; footprint 04_MyFoot_Passive:CP_EIA-3528-21_Kemet-B_HandSolder -> 04_MyFoot_Passive:CP_Elec_4x5.4; LCSC (none) -> C2895271
- C12, C18: value 10pF -> CG100J; footprint (none) -> 04_MyFoot_Passive:C_3216Metric; LCSC (none) -> C1883
- C2, C34, C6: value TAJB106K -> 10UF25V67RV; footprint 04_MyFoot_Passive:CP_EIA-3528-21_Kemet-B_HandSolder -> 04_MyFoot_Passive:CP_Elec_4x5.4; LCSC (none) -> C2895271
- C20: value CL475K -> CL21B475K; LCSC (none) -> C16194948
- C22: value CG101J -> CL21C101J; LCSC (none) -> C1790
- C24, C3, C59, C65: value CL106K -> CL31B106K; footprint 04_MyFoot_Passive:C_2012Metric -> 04_MyFoot_Passive:C_3216Metric; LCSC (none) -> C307369
- C25: value 104KC100V -> 0.1uF100V; footprint 04_MyFoot_Passive:C_2012Metric -> 04_MyFoot_Passive:C_Rect_W7.0mm_P15.00mm
- C26: value 10UF100V -> 10UF100V67RV; footprint 04_MyFoot_Passive:CP_EIA-3528-21_Kemet-B_HandSolder -> 04_MyFoot_Passive:CP_Elec_6.3x7.7; LCSC (none) -> C2895274
- C27: footprint 04_MyFoot_Passive:CP_EIA-3528-21_Kemet-B_HandSolder -> 04_MyFoot_Passive:CP_Radial_D16.0mm_P7.50mm
- C29, C8: value 47UF50V -> 47UF50V67RV; footprint 04_MyFoot_Passive:CP_EIA-3528-21_Kemet-B_HandSolder -> 04_MyFoot_Passive:CP_Elec_6.3x7.7; LCSC (none) -> C2887275
- C32, C35: LCSC (none) -> C157687
- C36, C41: value 0.1uF/100V -> 0.1uF100V; footprint (none) -> 04_MyFoot_Passive:C_Rect_W7.0mm_P15.00mm
- C37, C38, C43, C44: value 100nF -> CL31B104K; footprint (none) -> 04_MyFoot_Passive:C_3216Metric; LCSC (none) -> C1945
- C39, C40: LCSC (none) -> C24658
- C42: value 1uF/100V -> 1uF100V; footprint (none) -> 04_MyFoot_Passive:C_Rect_W7.0mm_P15.00mm
- C45: value 105J100V -> 1206B105K101NT; LCSC (none) -> C91151
- C46: value 223J100V -> 1206B223K101NT; LCSC (none) -> C48996
- C47, C48: value 225J100V -> CL31B225K; LCSC (none) -> C39619
- C49, C57: value 330J100V -> 1206CG331J101NT; LCSC (none) -> C20617886
- C50: value 220UF50V -> 220UF50V67RV; footprint 04_MyFoot_Passive:CP_EIA-3528-21_Kemet-B_HandSolder -> 04_MyFoot_Passive:CP_Elec_10x10.5; LCSC (none) -> C2887271
- C51: value 226J50V -> CL31A106K; LCSC (none) -> C13585
- C54, C58: value 103J100V -> 1206B103K; LCSC (none) -> C55077
- C55: value 102J100V -> 1206CG102J101NT; LCSC (none) -> C44911
- C56: value 101J100V -> 1206CG101J; LCSC (none) -> C1884
- C61, C63: value CL105K -> CL31B105K; footprint 04_MyFoot_Passive:C_2012Metric -> 04_MyFoot_Passive:C_3216Metric; LCSC (none) -> C13832
- C67, C68, C69, C70, C71: value B472K -> CL21B472K; LCSC (none) -> C50131
- D10, D11, D12, D13, D14, D15, D16, D7, D8: footprint 03_MyFoot_Active:D_MELF_Hand -> 03_MyFoot_Active:LL4148_MELF; LCSC (none) -> C84062
- D4, D5: value BAT54WS -> BAT54WSQ-7; footprint Diode_SMD:D_SOD-323 -> 03_MyFoot_Active:D_SOD-323_HandSoldering; LCSC (none) -> C171824
- D6: LCSC (none) -> C134447
- D9: value SM712_SOT23 -> SM712-LF-T7; LCSC (none) -> C2687124
- FB1: value FerriteBead -> CBG321609U; footprint (none) -> 04_MyFoot_Passive:R_3216Metric; LCSC (none) -> C74486
- FC1, FC2: value 470uF/63V -> 470UF63V; footprint (none) -> 04_MyFoot_Passive:CP_Radial_D12.5mm_P5.00mm
- IC1: footprint SOP65P640X110-21N -> 01_MyFoot_ICs:SOP65P640X110-21N; LCSC (none) -> C55575
- J1, J7: footprint SMW25002 -> 02_MyFoot_Connectors:SMW250_02P
- L1, L2, L4, L5, L6, L7, L8: footprint (none) -> 04_MyFoot_Passive:L_Radial_D10.0mm_P5.00mm
- L3: value Inductor -> 33uH; footprint (none) -> 04_MyFoot_Passive:L_Radial_D10.0mm_P5.00mm
- R1, R14, R2, R25, R39, R42, R44, R46, R48: value W8-J0103 -> W8J0103; LCSC (none) -> C25612
- R10, R17, R18: footprint (none) -> 04_MyFoot_Passive:R_Axial_2W_P20.32mm
- R11, R13: value FR-0747RL -> 0805FR-0747RL; LCSC (none) -> C114541
- R12, R19: value W4-J0103 -> 1812J103; footprint 04_MyFoot_Passive:R_2012Metric -> 04_MyFoot_Passive:R_4532Metric; LCSC (none) -> C2933913
- R15: value W8-J0104 -> 0805FR-07100K; LCSC (none) -> C96346
- R16, R9: value 1W-4.7 -> 25121WF470; footprint 04_MyFoot_Passive:R_2012Metric -> 04_MyFoot_Passive:R_6332Metric; LCSC (none) -> C474195
- R20, R21: value 10K -> W4F1002; footprint (none) -> 04_MyFoot_Passive:R_3216Metric; LCSC (none) -> C17902
- R22: value FR-0733RL -> 0805FR-0733RL; LCSC (none) -> C126353
- R23: value W4-J0123 -> W4J0123; footprint 04_MyFoot_Passive:R_2012Metric -> 04_MyFoot_Passive:R_3216Metric; LCSC (none) -> C2771295
- R24: value W4-J0334 -> W4J0334; LCSC (none) -> C25659
- R26: value 1W-F100 -> FRL2512FR047TS-47mohm; footprint Resistor_SMD:R_2512_6332Metric_Pad1.40x3.35mm_HandSolder -> 04_MyFoot_Passive:R_2512_6332Metric; LCSC (none) -> C7467449
- R27: value W4-F1102 -> W4F7502; footprint 04_MyFoot_Passive:R_2012Metric -> 04_MyFoot_Passive:R_3216Metric; LCSC (none) -> C17986
- R28: value W4-F1102 -> W4F9102; footprint 04_MyFoot_Passive:R_2012Metric -> 04_MyFoot_Passive:R_3216Metric; LCSC (none) -> C17981
- R29: value W4-J0223 -> W4J0223; footprint 04_MyFoot_Passive:R_2012Metric -> 04_MyFoot_Passive:R_3216Metric; LCSC (none) -> C25654
- R3, R4: value 200 -> AR06CTC0500; footprint (none) -> 04_MyFoot_Passive:R_3216Metric; LCSC (none) -> C5266090
- R30: value W4-F4992 -> W4F4992; footprint 04_MyFoot_Passive:R_2012Metric -> 04_MyFoot_Passive:R_3216Metric; LCSC (none) -> C18017
- R31: value W4-J0333 -> W4J0333; footprint 04_MyFoot_Passive:R_2012Metric -> 04_MyFoot_Passive:R_3216Metric; LCSC (none) -> C25660
- R32: value W4-J0100 -> W4J0100; footprint 04_MyFoot_Passive:R_2012Metric -> 04_MyFoot_Passive:R_3216Metric; LCSC (none) -> C25349
- R33: value W4-F1501 -> W4F4991; footprint 04_MyFoot_Passive:R_2012Metric -> 04_MyFoot_Passive:R_3216Metric; LCSC (none) -> C57609
- R34: value W4-F1501 -> W4F1002; footprint 04_MyFoot_Passive:R_2012Metric -> 04_MyFoot_Passive:R_3216Metric; LCSC (none) -> C17902
- R35: value W4-F2701 -> W4F8871; footprint 04_MyFoot_Passive:R_2012Metric -> 04_MyFoot_Passive:R_3216Metric; LCSC (none) -> C55354
- R36, R40: value W8-J0431 -> W8J0431; LCSC (none) -> C54672
- R37: value W4-J0121 -> W4J0121; footprint 04_MyFoot_Passive:R_2012Metric -> 04_MyFoot_Passive:R_3216Metric; LCSC (none) -> C25351
- R38, R41, R43, R45, R47: value W4-J0472 -> W4J0472; LCSC (none) -> C26043
- R5, R6, R7, R8: value 200 -> W4F4700; footprint (none) -> 04_MyFoot_Passive:R_3216Metric; LCSC (none) -> C4502
- SW1: value SW_Push -> TS-1088; footprint (none) -> 06_MyFoot_Mechanical:SW_SPST_TS-1088-xR025; LCSC (none) -> C455280
- SW2: value SW_DIP_x02 -> DSHP02T; footprint (none) -> 06_MyFoot_Mechanical:CHS-02B_W7.62mm_P1.27mm; LCSC (none) -> C40735
- U1: footprint Package_TO_SOT_SMD:SOT-223-3_TabPin2 -> 01_MyFoot_ICs:SOT-223-3_TabPin2; LCSC (none) -> C6186
- U10, U11, U12, U6, U9: value TLP185 -> TLP185GB-S; LCSC (none) -> C388375
- U2: value UCC21520DW -> UCC21520DWR; footprint Package_SO:SOIC-16W_7.5x10.3mm_P1.27mm -> 01_MyFoot_ICs:SOIC-16W_7.5x10.3mm_P1.27mm; LCSC (none) -> C601651
- U3: LCSC (none) -> C529413
Connections:
- net +15VA: now also DCDC1.4 (+Vout)
- net +15VB: now also DCDC2.4 (+Vout); no longer R12.1
- net +24V: now also DCDC1.2 (+Vin), DCDC2.2 (+Vin), J2.3 (Pin_3)
- net +3.3V: now also D1.2 (A), J3.1 (Pin_1), J3.7 (Pin_7), J5.1 (Pin_1), J6.14 (Pin_14), J6.16 (Pin_16), U4.3 (V+), U5.8 (VCC)
- net +48V: now also J2.1 (Pin_1)
- net +5V: now also J2.5 (Pin_5), J3.8 (Pin_8), J6.17 (Pin_17), J6.19 (Pin_19), U7.9 (COM), U8.9 (COM)
- net +VBUS: now also Q1.2 (D), U4.5 (-)
- net ADC1_IN1: now also D17.1 (K), R49.2; no longer C43.2, D4.1 (K), R20.2
- net ADC1_IN2: now also D18.1 (K), R50.2; no longer C44.2, D5.1 (K), R21.2
- net ADC2_IN3: now also U4.6
- net BCD_BIT1: now also J8.21 (Pin_21)
- net BCD_BIT2: now also J8.20 (Pin_20)
- net BCD_BIT3: now also J8.19 (Pin_19)
- net BZ_OUT: now also J6.12 (Pin_12)
- net CLK_LCD: now also J6.13 (Pin_13)
- net CLK_LED: now also J6.15 (Pin_15)
- net D0: now also J6.1 (Pin_1)
- net D1: now also J6.3 (Pin_3)
- net D2: now also J6.5 (Pin_5)
- net D3: now also J6.7 (Pin_7)
- net D4: now also J6.9 (Pin_9)
- net D5: now also J6.11 (Pin_11)
- net DE_RS485: now also U5.3 (DE)
- net DOWN: now also J6.8 (Pin_8)
- net DTR: now also J4.1 (Pin_1)
- net GND: now also C52.1, R34.1, D1.1 (K), D17.2 (A), D18.2 (A), DCDC1.1 (-Vin), DCDC2.1 (-Vin), H1.1, H2.1, J2.4 (Pin_4), J2.6 (Pin_6), J3.3 (Pin_3), J3.9 (Pin_9), J4.6 (Pin_6), J5.3 (Pin_3), J6.18 (Pin_18), J6.20 (Pin_20), J8.17 (Pin_17), J8.24 (Pin_24), R51.1, T1.4, U4.1 (REF), U4.2 (GND), U5.5 (GND), U7.8 (GND), U8.8 (GND)
- net GNDA: now also R12.1, DCDC1.3 (-Vout), Q1.3 (S), Q2.2 (D), T1.1
- net GNDB: now also DCDC2.3 (-Vout), J2.2 (Pin_2), Q2.3 (S), R51.2; no longer C52.1, R34.1
- net GOING: now also U8.2 (I2)
- net GOING_A: now also J8.3 (Pin_3)
- net GOING_C: now also J8.4 (Pin_4)
- net HIGH_ALARM: now also U8.3 (I3)
- net HIGH_ALARM_A: now also J8.5 (Pin_5)
- net HIGH_ALARM_C: now also J8.6 (Pin_6)
- net LC_REL1: now also U7.4 (I4)
- net LC_REL2: now also U7.3 (I3)
- net LC_REL3: now also U7.2 (I2)
- net LC_REL4: now also U7.1 (I1)
- net LOW_ALARM: now also U8.1 (I1)
- net LOW_ALARM_A: now also J8.1 (Pin_1)
- net LOW_ALARM_C: now also J8.2 (Pin_2)
- net MODE: now also J6.4 (Pin_4)
- net NRST: now also D1.3 (K), J3.10 (Pin_10)
- net REMOTE: now also J8.18 (Pin_18)
- net SENSOR: now also J8.25 (Pin_25)
- net SET: now also J6.10 (Pin_10)
- net START_STOP: now also J6.2 (Pin_2)
- net SWCLK: now also J3.4 (Pin_4)
- net SWDIO: now also J3.2 (Pin_2)
- net TD_ALARM: now also U8.4 (I4)
- net TD_ALARM_A: now also J8.11 (Pin_11)
- net TD_ALARM_C: now also J8.12 (Pin_12)
- net TOTAL_ALARM: now also U8.5 (I5)
- net TOTAL_ALARM_A: now also J8.13 (Pin_13)
- net TOTAL_ALARM_C: now also J8.14 (Pin_14)
- net UP: now also J6.6 (Pin_6)
- net USART1_RX: now also J4.3 (Pin_3)
- net USART1_TX: now also J4.2 (Pin_2)
- net USART2_RX: now also U5.1 (RO)
- net USART2_TX: now also U5.4 (DI)
- net /RE_RS485: now also U5.2 (~{RE})
- net at D16.2 (A), K9.16 (COIL-): now also U7.13 (O4)
- net at D13.2 (A), K6.16 (COIL-): now also U7.14 (O3)
- net at D11.2 (A), K4.16 (COIL-): now also U7.15 (O2)
- net at D7.2 (A), K1.16 (COIL-): now also U7.16 (O1)
- net at D9.1 (A1), D9.2 (A2), J7.1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: now also U5.6 (A)
- net at D9.3 (common), J7.2, R40.2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: now also U5.7 (B)
- net at D15.2 (A), K8.1 (-): now also U8.12 (O5)
- net at R16.1, R19.2: now also D3.2 (A2), Q2.1 (G)
- net at C18.2, L1.1, L2.1: now also T2.2
- net at R16.2, U2.10 (OUTB): now also D3.1 (A1)
- net at C50.1, C51.2, IC1.12 (OUT)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: now also U4.4 (+)
- net at R3.2, R5.2, R6.2: now also T2.3
- net at R4.2, R7.2, R8.2: now also T2.4
- net at C12.2: now also T1.3, T2.1
- net at R9.2, U2.15 (OUTA): now also D2.1 (A1)
- net at R12.2, R9.1: now also D2.2 (A2), Q1.1 (G)
- net at D14.2 (A), K7.1 (-): now also U8.13 (O4)
- net at R25.2, U3.61 (PB8): now also J5.2 (Pin_2)
- net at C35.2, U3.6 (PF1): now also Y1.1
- net at C36.1, C41.2, FC1.2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: now also T1.2
- net at C32.2, U3.5 (PF0): now also Y1.2
- net at D12.2 (A), K5.1 (-): now also U8.14 (O3)
- net at D10.2 (A), K3.1 (-): now also U8.15 (O2)
- net at D8.2 (A), K2.1 (-): now also U8.16 (O1)
- new net: C44.2, D5.1 (K), R21.2, R50.1
- new net: C43.2, D4.1 (K), R20.2, R49.1
- no-connect marks 0 -> 38
Other:
- note added: "10(ID)16(OD)SN-02HT CT 1:20T"
- note added: "PL-F2 OUTPUT TRANS 20(OD)10(ID) 6T:12T LITZ 0.2mm ENAMEL"
- moved on the sheet: C21, C55, C57, R20, R31, U1
