File: kicad/ELSONIC/Multi_Mega_Main_V2/Multi_Mega_Main_V2.kicad_sch (KiCad schematic)
At the start: 193 parts, among them IC1 LM5005MHX_NOPB, J1 SMW250-02P, J2 Screw_Terminal_01x06, J3 ARM_SWD_10, J4 Conn_01x06_HEADERPIN, J5 Conn_01x03, J6 Conn_02x10_Odd_Even, J7 SMW250-02P, J8 Conn_02x13_Odd_Even, K1 G6A274, K2 PA1A_5V, K3 PA1A_5V, K4 G6A274, K5 PA1A_5V, K6 G6A274, K7 PA1A_5V, K8 PA1A_5V, K9 G6A274, Q1 STD25N10F7, Q2 STD25N10F7, SW1 TS-1088, SW2 DSHP02T, T1 TOROID_OUTPUT_OD20_T6T12, T2 TOROID_CT_OD16_T1T20, U1 AMS1117-3.3, U10 TLP185GB-S, U11 TLP185GB-S, U12 TLP185GB-S, U2 UCC21520DWR, U3 STM32G474RBT6, U4 INA190A3IDCKR, U5 MAX3485ESA, U6 TLP185GB-S, U7 ULN2003ADR, U8 ULN2003ADR, U9 TLP185GB-S, Y1 X49SM8M

Commit message: chore: sync remaining hardware design assets
Parts:
- C42: value 1uF100V -> 0.1uF100V
- L2: value 3.9uH -> 4.7uH
- L4: value 1.5uH -> 1.0uH
- L6: value 2.7uH -> 2.2uH
- R24: footprint 04_MyFoot_Passive:R_2012Metric -> 04_MyFoot_Passive:R_3216Metric
- R27: value W4F7502 -> W4F7502(120k)
- R34: value W4F1002 -> W4F1002(5k)
- T1: value TOROID_OUTPUT_OD20_T6T12 -> TOROID_OUTPUT_OD20_T6T12(T7:T24)
Other:
- note added: "10(ID)16(OD)SN-02HT CT 1:20T(2:15)"
- note removed: "10(ID)16(OD)SN-02HT CT 1:20T"
Changed lines of the file:
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@@
 		)
 	)
-	(text "10(ID)16(OD)SN-02HT CT 1:20T"
+	(text "10(ID)16(OD)SN-02HT CT 1:20T(2:15)"
 		(exclude_from_sim no)
 		(at 501.904 30.226 0)
@@
 			)
 		)
-		(property "Value" "W4F7502"
+		(property "Value" "W4F7502(120k)"
 			(at 428.244 143.51 0)
 			(show_name no)
@@
 			)
 		)
-		(property "Footprint" "04_MyFoot_Passive:R_2012Metric"
+		(property "Footprint" "04_MyFoot_Passive:R_3216Metric"
 			(at 296.926 129.286 90)
 			(hide yes)
@@
 			)
 		)
-		(property "Value" "3.9uH"
+		(property "Value" "4.7uH"
 			(at 524.51 26.67 90)
 			(show_name no)
@@
 			)
 		)
-		(property "Value" "W4F1002"
+		(property "Value" "W4F1002(5k)"
 			(at 451.866 157.734 0)
 			(show_name no)
@@
 			)
 		)
-		(property "Value" "1.5uH"
+		(property "Value" "1.0uH"
 			(at 357.632 251.714 90)
 			(show_name no)
@@
 			)
 		)
-		(property "Value" "2.7uH"
+		(property "Value" "2.2uH"
 			(at 356.87 297.18 90)
 			(show_name no)
@@
 			)
 		)
-		(property "Value" "TOROID_OUTPUT_OD20_T6T12"
+		(property "Value" "TOROID_OUTPUT_OD20_T6T12(T7:T24)"
 			(at 453.39 82.55 0)
 			(show_name no)
@@
 			)
 		)
-		(property "Value" "1uF100V"
+		(property "Value" "0.1uF100V"
 			(at 442.468 103.632 0)
 			(show_name no)

Commit message: feat: update ultrasonic controller and board design
Connections:
- net GND: now also D9.3 (common)
- net at D9.1 (A1), J7.1, R36.1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: no longer D9.2 (A2)
- net at J7.2, R40.2, SW2.4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: now also D9.2 (A2); no longer D9.3 (common)
Other:
- note added: "560R~1K"
Changed lines of the file:
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@@
 		)
 	)
+	(text "560R~1K "
+		(exclude_from_sim no)
+		(at 461.772 263.144 0)
+		(effects
+			(font
+				(size 1.27 1.27)
+			)
+		)
+	)
+	(text "560R~1K "
+		(exclude_from_sim no)
+		(at 461.518 234.696 0)
+		(effects
+			(font
+				(size 1.27 1.27)
+			)
+		)
+	)
 	(text "10(ID)16(OD)SN-02HT CT 1:20T(2:15)"
 		(exclude_from_sim no)
@@
 	)
 	(junction
+		(at 472.44 255.27)
+		(diameter 0)
+		(color 0 0 0 0)
+	)
+	(junction
 		(at 350.52 22.86)
 		(diameter 0)
@@
 	)
 	(junction
-		(at 457.2 246.38)
-		(diameter 0)
-		(color 0 0 0 0)
-	)
-	(junction
 		(at 444.5 135.89)
 		(diameter 0)
@@
 	)
 	(junction
-		(at 464.82 241.3)
-		(diameter 0)
-		(color 0 0 0 0)
-	)
-	(junction
 		(at 548.64 101.6)
 		(diameter 0)
@@
 	)
 	(junction
-		(at 472.44 233.68)
-		(diameter 0)
-		(color 0 0 0 0)
-	)
-	(junction
 		(at 309.88 167.64)
 		(diameter 0)
@@
 		(color 0 0 0 0)
 	)
+	(junction
+		(at 472.44 233.68)
+		(diameter 0)
+		(color 0 0 0 0)
+	)
 	(no_connect
 		(at 181.61 74.93)
@@
 	(wire
 		(pts
-			(xy 472.44 236.22) (xy 472.44 233.68)
-		)
-		(stroke
-			(width 0)
-			(type default)
-		)
-	)
-	(wire
-		(pts
 			(xy 123.19 50.8) (xy 123.19 53.34)
 		)
@@
 	(wire
 		(pts
-			(xy 491.49 255.27) (xy 457.2 255.27)
+			(xy 491.49 255.27) (xy 472.44 255.27)
 		)
 		(stroke
@@
 	(wire
 		(pts
+			(xy 472.44 254) (xy 472.44 255.27)
+		)
+		(stroke
+			(width 0)
+			(type default)
+		)
+	)
+	(wire
+		(pts
 			(xy 487.68 106.68) (xy 490.22 106.68)
 		)
@@
 	(wire
 		(pts
-			(xy 464.82 254) (xy 464.82 241.3)
-		)
-		(stroke
-			(width 0)
-			(type default)
-		)
-	)
-	(wire
-		(pts
 			(xy 83.82 236.22) (xy 83.82 237.49)
 		)
@@
 	(wire
 		(pts
+			(xy 472.44 233.68) (xy 472.44 236.22)
+		)
+		(stroke
+			(width 0)
+			(type default)
+		)
+	)
+	(wire
+		(pts
 			(xy 229.87 314.96) (xy 229.87 322.58)
 		)
@@
 	(wire
 		(pts
+			(xy 468.63 245.11) (xy 463.55 245.11)
+		)
+		(stroke
+			(width 0)
+			(type default)
+		)
+	)
+	(wire
+		(pts
 			(xy 288.29 54.61) (xy 288.29 57.15)
 		)
@@
 	(wire
 		(pts
-			(xy 468.63 245.11) (xy 457.2 245.11)
+			(xy 303.53 167.64) (xy 309.88 167.64)
 		)
 		(stroke
@@
 	(wire
 		(pts
-			(xy 303.53 167.64) (xy 309.88 167.64)
+			(xy 478.79 140.97) (xy 483.87 140.97)
 		)
 		(stroke
@@
 	(wire
 		(pts
-			(xy 478.79 140.97) (xy 483.87 140.97)
+			(xy 373.38 269.24) (xy 373.38 270.51)
 		)
 		(stroke
@@
 	(wire
 		(pts
-			(xy 373.38 269.24) (xy 373.38 270.51)
+			(xy 463.55 245.11) (xy 463.55 246.38)
 		)
 		(stroke
@@
 	(wire
 		(pts
+			(xy 472.44 255.27) (xy 457.2 255.27)
+		)
+		(stroke
+			(width 0)
+			(type default)
+		)
+	)
+	(wire
+		(pts
 			(xy 93.98 364.49) (xy 99.06 364.49)
 		)
@@
 	(wire
 		(pts
-			(xy 472.44 233.68) (xy 464.82 233.68)
+			(xy 464.82 233.68) (xy 472.44 233.68)
 		)
 		(stroke
@@
 	(wire
 		(pts
+			(xy 472.44 233.68) (xy 491.49 233.68)
+		)
+		(stroke
+			(width 0)
+			(type default)
+		)
+	)
+	(wire
+		(pts
 			(xy 389.89 90.17) (xy 389.89 85.09)
 		)
@@
 	(wire
 		(pts
-			(xy 457.2 245.11) (xy 457.2 246.38)
-		)
-		(stroke
-			(width 0)
-			(type default)
-		)
-	)
-	(wire
-		(pts
 			(xy 214.63 360.68) (xy 203.2 360.68)
 		)
@@
 	(wire
 		(pts
-			(xy 491.49 233.68) (xy 472.44 233.68)
-		)
-		(stroke
-			(width 0)
-			(type default)
-		)
-	)
-	(wire
-		(pts
 			(xy 463.55 135.89) (xy 464.82 135.89)
 		)
@@
 	(wire
 		(pts
-			(xy 472.44 254) (xy 464.82 254)
-		)
-		(stroke
-			(width 0)
-			(type default)
-		)
-	)
-	(wire
-		(pts
 			(xy 496.57 41.91) (xy 496.57 49.53)
 		)
@@
 		(lib_id "Diode:SM712_SOT23")
 		(at 472.44 245.11 270)
-		(mirror x)
 		(unit 1)
 		(body_style 1)
@@
 		(dnp no)
 		(property "Reference" "D9"
-			(at 474.98 243.84 90)
+			(at 474.98 246.38 90)
 			(show_name no)
 			(do_not_autoplace no)
@@
 		)
 		(property "Value" "SM712-LF-T7"
-			(at 474.98 246.38 90)
+			(at 474.98 243.84 90)
 			(show_name no)
 			(do_not_autoplace no)
@@
 		)
 		(property "Datasheet" ""
-			(at 472.44 248.92 0)
+			(at 472.44 241.3 0)
 			(hide yes)
 			(show_name no)
@@
 					(unit 1)
 				)
+			)
+		)
+	)
+	(symbol
+		(lib_id "power:GND")
+		(at 463.55 246.38 0)
+		(unit 1)
+		(body_style 1)
+		(exclude_from_sim no)
+		(in_bom yes)
+		(on_board yes)
+		(in_pos_files yes)
+		(dnp no)
+		(property "Reference" "#PWR0145"
+			(at 463.55 252.73 0)
+			(hide yes)
+			(show_name no)
+			(do_not_autoplace no)
+			(effects
+				(font
+					(size 1.27 1.27)
+				)
+			)
+		)
+		(property "Value" "GND"
+			(at 467.106 248.158 0)
+			(show_name no)
+			(do_not_autoplace no)
+			(effects
+				(font
+					(size 1.27 1.27)
+				)
+			)
+		)
+		(property "Footprint" ""
+			(at 463.55 246.38 0)
+			(hide yes)
+			(show_name no)
+			(do_not_autoplace no)
+			(effects
+				(font
+					(size 1.27 1.27)
+				)
+			)
+		)
+		(property "Datasheet" ""
+			(at 463.55 246.38 0)
+			(hide yes)
+			(show_name no)
+			(do_not_autoplace no)
+			(effects
+				(font
+					(size 1.27 1.27)
+				)
+			)
+		)
+		(property "Description" "Power symbol creates a global label with name \"GND\" , ground"
+			(at 463.55 246.38 0)
+			(hide yes)
+			(show_name no)
+			(do_not_autoplace no)
+			(effects
+				(font
+					(size 1.27 1.27)
+				)
+			)
+		)
+		(pin "1"
+		)
+		(instances
+			(project "Multi_Mega_Main_V2"
+				(path "/846747d2-d9a3-4232-803f-01fc97424ea2"
+					(reference "#PWR0145")
+					(unit 1)
+				)
