File: kicad/ELSONIC/Multi_Mega_Display_V2/Multi_Mega_Display_V2.kicad_sch (KiCad schematic)
At the start: 48 parts, among them J2 Conn_01x01, J3 Conn_01x01, J4 Conn_01x01, J5 Conn_01x01, J6 Conn_02x10_Odd_Even, Q1 KRC105S, U1 74HCT574PWR, U2 74HCT574PWR

Commit message: chore: sync remaining hardware design assets
Other:
- note added: "D0:D1:NORMAL D1:D2:H/L SET D2:D3:8POWER D3:D4:REMOTE D4:D5:EXT D5:D6:TXRX"
Changed lines of the file:
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@@
 	(generator_version "10.0")
 	(paper "A3")
+	(text "D0:D1:NORMAL D1:D2:H/L SET D2:D3:8POWER D3:D4:REMOTE D4:D5:EXT D5:D6:TXRX"
+		(exclude_from_sim no)
+		(at 289.814 149.606 0)
+		(effects
+			(font
+				(size 1.27 1.27)
+			)
+		)
+	)
 	(junction
 		(at 204.47 200.66)
