File: kicad/ELSONIC/POWER_BD_SV5/POWER_BD_SV5.kicad_pcb (KiCad board)
At the start: 2 copper layers, 150 x 98 mm, 99 parts, among them J2 SMW250-06P, J3 SMW250-02P, T1 EI2811BP, T2 EER28, U1 ICE3BR0665J, U2 H11AA1, U3 PC817, U4 ATTINY85-20PU_1, U5 MOC3021M, U6 LM7805_TO220

Commit message: chore: sync remaining hardware design assets
Parts:
- C10: footprint 04_MyFoot_Passive:CP_Radial_D5.0mm_P2.00mm -> 04_MyFoot_Passive:CP_Elec_6.3x5.4
- C16, C17, C18: footprint 04_MyFoot_Passive:C_Disc_D4.7mm_P5.00mm -> 04_MyFoot_Passive:C_3216Metric
- C29: footprint 04_MyFoot_Passive:CP_Radial_D6.3mm_P2.50mm -> 04_MyFoot_Passive:CP_Elec_6.3x7.7
- C7: footprint 04_MyFoot_Passive:C_Disc_D6.0mm_P5.00mm -> 04_MyFoot_Passive:C_3216Metric
- D2, D3: footprint 03_MyFoot_Active:Diode_P10.16mm -> 03_MyFoot_Active:D_SMA
- D4: value 1N5251 -> BZT52C22; footprint 03_MyFoot_Active:ZENER_0_5W_P7.62mm_Hori -> 03_MyFoot_Active:D_SOD-123
- L1, L2, L3: footprint 04_MyFoot_Passive:L_Radial_D7.5mm_P3.50mm -> 04_MyFoot_Passive:L_Sumida_CDMC6D28_7.25x6.5mm
- LED1, LED2: value LED_SMD -> LED_SMD_KT_0805R
- R12: value 820R -> 820R/F
- R14, R15, R16: footprint 04_MyFoot_Passive:R_3216Metric -> 04_MyFoot_Passive:R_4532Metric
- R17: value 68K -> 68K/F
- R18: value 1K/F -> 2K/F
- R19: value 40K/F -> 39K/F
- R2: value 1.2K -> 2.2K
- R24, R25, R3, R4: footprint 04_MyFoot_Passive:R_Axial_1W_P14.6mm -> 04_MyFoot_Passive:R_6332Metric
- R6: value 10K -> 4.7K
- U2: value H11AA1 -> EL354N; footprint 01_MyFoot_ICs:DIP-6_W7.62mm -> 01_MyFoot_ICs:SOIC-4_EL354_P2.54mm
- U3: value PC817 -> TLP785(GB-TP6F); footprint 01_MyFoot_ICs:DIP-4_W7.62mm_Socket -> 01_MyFoot_ICs:SOP-4_7.5x4.1mm_P2.54mm
- U5: value MOC3021M -> MOC3021SM; footprint 01_MyFoot_ICs:DIP-6_W7.62mm -> 01_MyFoot_ICs:SOIC-6_P2.54mm
- U6: footprint 01_MyFoot_ICs:TO220_P2.54mm -> 01_MyFoot_ICs:TO-252-2
- VR1: value TL431A -> TL431DBZ; footprint 01_MyFoot_ICs:TO92_P2.5mm -> 01_MyFoot_ICs:SOT-23-3
- moved D4 16.8 mm to (69.5, -56.0)
- moved C30 8.71 mm to (26.5, -16.5)
- moved C18 5.70 mm to (45.5, -20.5)
- moved R16 5.39 mm to (45.0, -27.0), turned to -90 degrees
- moved C28 4.14 mm to (19.5, -16.5)
- moved D3 3.89 mm to (61.0, -55.5), turned to 180 degrees
- moved R25 3.20 mm to (143.5, -13.0)
- moved R4 2.90 mm to (65.0, -63.5)
- moved R3 2.81 mm to (70.0, -63.5)
- moved VR1 2.00 mm to (53.5, -25.0), turned to 180 degrees
- moved U6 1.71 mm to (24.0, -28.0)
- moved D2 1.71 mm to (67.0, -92.0)
- moved C7 1.63 mm to (68.0, -82.0)
- moved L3 1.52 mm to (48.0, -13.0)
- moved C10 1.50 mm to (71.5, -46.0)
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- renumbered F2 to F1, H4 to H2, H2 to H3, H3 to H4
Connections:
- net Net-(T1-SB) renamed /AC12V
- C15 pad 1: Net-(C15-Pad1) -> Net-(VR1-K)
- C19 pad 2: Net-(C19-Pad2) -> Net-(VR1-REF)
- LED1 pad 1: GND -> Net-(LED1-A)
- LED1 pad 2: Net-(LED1-A) -> GND
- LED2 pad 1: GND -> Net-(LED2-A)
- LED2 pad 2: Net-(LED2-A) -> GND
- R12 pad 2: Net-(C15-Pad1) -> Net-(VR1-K)
- R13 pad 1: Net-(C15-Pad1) -> Net-(VR1-K)
- R17 pad 1: Net-(C15-Pad1) -> Net-(VR1-K)
- R19 pad 1: Net-(C19-Pad2) -> Net-(VR1-REF)
- R20 pad 2: Net-(C19-Pad2) -> Net-(VR1-REF)
- U2 pad 3: unconnected-(U2-Pad3) -> GND
- U2 pad 4: GND -> /ZVC
- VR1 pad 1: Net-(C19-Pad2) -> Net-(VR1-K)
- VR1 pad 2: GND -> Net-(VR1-REF)
- VR1 pad 3: Net-(C15-Pad1) -> GND
Routing:
- net GND: track 52.8 -> 91.2 mm, vias 2 -> 44
- net Net-(VR1-K): track 0.00 -> 33.1 mm, vias 0 -> 2
- net Net-(C15-Pad1): track 32.9 -> 0.00 mm, vias 1 -> 0
- net Net-(C19-Pad2): track 26.0 -> 0.00 mm
- net Net-(VR1-REF): track 0.00 -> 20.5 mm, vias 0 -> 2
- net Earth: track 207.3 -> 190.5 mm
- net Net-(D3-A): track 29.4 -> 38.4 mm, vias 0 -> 1
- net Net-(T2-N1): track 84.3 -> 75.6 mm
- net Net-(D4-K): track 17.4 -> 11.1 mm, vias 0 -> 2
- net +8V: track 38.5 -> 33.7 mm, vias 0 -> 1
- net Net-(R24-Pad1): track 9.49 -> 13.8 mm, vias 0 -> 2
- net Net-(D2-A): track 62.5 -> 66.1 mm
- net +5V: track 168.5 -> 171.9 mm
- net Net-(T2-N2): track 54.6 -> 51.7 mm
- net Net-(C31-Pad1): track 53.5 -> 56.1 mm
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Other:
- outline, holes or cut-outs redrawn
- board text added: "POWER_BD_SV5.0"
- board text removed: "POWER_BD_SV2.0"
