File: kicad/ELSONIC/POWER_BD_SV5/POWER_BD_SV5.kicad_sch (KiCad schematic)
At the start: 99 parts, among them J2 SMW250-06P, J3 SMW250-02P, T1 EI2811BP, T2 EER28, U1 ICE3BR0665J, U2 H11AA1, U3 PC817, U4 ATTINY85-20PU_1, U5 MOC3021M, U6 LM7805_TO220

Commit message: chore: sync remaining hardware design assets
Parts:
- removed LED1, LED2: LED_SMD, 03_MyFoot_Active:LED_2012Metric, symbol 03_MyLib_Active:LED_SMD
- removed U2: H11AA1, 01_MyFoot_ICs:DIP-6_W7.62mm, symbol 01_MyLib_ICs:H11AA1
- removed VR1: TL431A, 01_MyFoot_ICs:TO92_P2.5mm, symbol 01_MyLib_ICs:TL431A
- added LED1, LED2: LED_SMD_KT_0805R, 03_MyFoot_Active:LED_2012Metric, symbol 03_MyLib_Active:LED_SMD_KT_0805R
- added U2: EL354N, 01_MyFoot_ICs:SOIC-4_EL354_P2.54mm, symbol 01_MyLib_ICs:PC817X3NSZ1B
- added VR1: TL431DBZ, 01_MyFoot_ICs:SOT-23-3, symbol 01_MyLib_ICs:TL431DBZ
- C10: footprint 04_MyFoot_Passive:CP_Radial_D5.0mm_P2.00mm -> 04_MyFoot_Passive:CP_Elec_6.3x5.4; LCSC (none) -> C970678
- C11, C13: LCSC (none) -> C76663
- C15, C6: LCSC (none) -> C1941
- C16, C17, C18: footprint 04_MyFoot_Passive:C_Disc_D4.7mm_P5.00mm -> 04_MyFoot_Passive:C_3216Metric
- C19: LCSC (none) -> C1857
- C29: footprint 04_MyFoot_Passive:CP_Radial_D6.3mm_P2.50mm -> 04_MyFoot_Passive:CP_Elec_6.3x7.7; LCSC (none) -> C2992606
- C7: footprint 04_MyFoot_Passive:C_Disc_D6.0mm_P5.00mm -> 04_MyFoot_Passive:C_3216Metric; LCSC (none) -> C9192
- C8: LCSC (none) -> C1868
- D2, D3: footprint 03_MyFoot_Active:Diode_P10.16mm -> 03_MyFoot_Active:D_SMA; LCSC (none) -> C81191
- D4: value 1N5251 -> BZT52C22; footprint 03_MyFoot_Active:ZENER_0_5W_P7.62mm_Hori -> 03_MyFoot_Active:D_SOD-123; LCSC (none) -> C2108
- L1, L2, L3: footprint 04_MyFoot_Passive:L_Radial_D7.5mm_P3.50mm -> 04_MyFoot_Passive:L_Sumida_CDMC6D28_7.25x6.5mm; LCSC C237927 -> C436542
- R10: LCSC (none) -> C17936
- R12: LCSC (none) -> C17984
- R13: LCSC (none) -> C17891
- R14, R15, R16: footprint 04_MyFoot_Passive:R_3216Metric -> 04_MyFoot_Passive:R_4532Metric; LCSC C25349 -> C2933875
- R17: LCSC (none) -> C25834
- R18: LCSC (none) -> C17944
- R19: LCSC (none) -> C18008
- R2: value 1.2K -> 2.2K/F; LCSC (none) -> C17948
- R20: LCSC (none) -> C17902
- R21: LCSC (none) -> C26035
- R22: LCSC (none) -> C26038
- R23: LCSC (none) -> C17957
- R24: footprint 04_MyFoot_Passive:R_Axial_1W_P14.6mm -> 04_MyFoot_Passive:R_6332Metric; LCSC (none) -> C38808
- R25: footprint 04_MyFoot_Passive:R_Axial_1W_P14.6mm -> 04_MyFoot_Passive:R_6332Metric; LCSC (none) -> C37457
- R27: LCSC (none) -> C25348
- R3, R4: footprint 04_MyFoot_Passive:R_Axial_1W_P14.6mm -> 04_MyFoot_Passive:R_6332Metric
- R6: value 10K -> 4.7K; LCSC C1489 -> C17936
- R9: LCSC (none) -> C17901
- U1: LCSC C152412 -> (none)
- U3: value PC817 -> TLP785(GB-TP6F); footprint 01_MyFoot_ICs:DIP-4_W7.62mm_Socket -> 01_MyFoot_ICs:SOP-4_7.5x4.1mm_P2.54mm; LCSC C41807 -> C45445
- U5: value MOC3021M -> MOC3021SM; footprint 01_MyFoot_ICs:DIP-6_W7.62mm -> 01_MyFoot_ICs:SOIC-6_P2.54mm
- U6: footprint 01_MyFoot_ICs:TO220_P2.54mm -> 01_MyFoot_ICs:TO-252-2
- renumbered F2 to F1, H4 to H2, H2 to H3, H3 to H4
Connections:
- net GND: now also LED1.2 (K), LED2.2 (K), U2.3, VR1.3 (A)
- net ZVC: now also U2.4
- net at C19.2, R19.1, R20.2: now also VR1.2 (REF)
- net at R21.2: now also LED1.1 (A)
- net at R2.2: now also U2.1
- net at T1.3 (SA): now also U2.2
- net at C15.1, R12.2, R13.1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: now also VR1.1 (K)
- net at R22.1: now also LED2.1 (A)
- no-connect marks 8 -> 6
Other:
- moved on the sheet: C8, R2, R6, T1
