File: kicad/ELSONIC/Multi_Mega_Main_V3/Multi_Mega_Main_V3.kicad_pcb (KiCad board)
At the start: 2 copper layers, 200 x 150 mm, 193 parts, among them IC1 LM5005MHX_NOPB, J1 SMW250-02P, J2 Screw_Terminal_01x06, J3 ARM_SWD_10, J4 Conn_01x06_HEADERPIN, J5 Conn_01x03, J6 Conn_02x10_Odd_Even, J7 SMW250-02P, J8 Conn_02x13_Odd_Even, K1 G6A274, K2 PA1A_5V, K3 PA1A_5V, K4 G6A274, K5 PA1A_5V, K6 G6A274, K7 PA1A_5V, K8 PA1A_5V, K9 G6A274, Q1 STD25N10F7, Q2 STD25N10F7, SW1 TS-1088, SW2 DSHP02T, T1 TOROID_OUTPUT_OD20_T6T12, T2 TOROID_CT_OD16_T1T20, U1 AMS1117-3.3, U10 TLP185GB-S, U11 TLP185GB-S, U12 TLP185GB-S, U2 UCC21520DWR, U3 STM32G474RBT6, U4 INA190A3IDCKR, U5 MAX3485ESA, U6 TLP185GB-S, U7 ULN2003ADR, U8 ULN2003ADR, U9 TLP185GB-S, Y1 X49SM8M

Commit message: feat: update ultrasonic controller and board design
Parts:
- added IC2: L7987TR, 01_MyFoot_ICs:SOP65P640X120-17N, F.Cu at (225.4, -51.1)
- added L9: 33uH, 04_MyFoot_Passive:L_Radial_D10.0mm_P5.00mm, F.Cu at (226.7, -60.4)
- added R52: W4F7502(200k), 04_MyFoot_Passive:R_3216Metric, F.Cu at (217.8, -64.5)
- added R53: 5K, 04_MyFoot_Passive:R_3216Metric, F.Cu at (217.8, -61.1)
- added R54: W4F9102, 04_MyFoot_Passive:R_3216Metric, F.Cu at (217.8, -57.8)
- added R55: W4F1002(5k), 04_MyFoot_Passive:R_3216Metric, F.Cu at (217.8, -54.4)
- added R56: 22K, 04_MyFoot_Passive:R_3216Metric, F.Cu at (217.8, -51.1)
- added R57: W8J0103, 04_MyFoot_Passive:R_2012Metric, F.Cu at (232.2, -53.1)
- added R58: W8J0103, 04_MyFoot_Passive:R_2012Metric, F.Cu at (232.2, -50.2)
- C42: value 1uF100V -> 0.1uF100V
- L2: value 3.9uH -> 4.7uH
- L4: value 1.5uH -> 1.0uH
- L6: value 2.7uH -> 2.2uH
- R12, R19: value 1812J103 -> 1812J222
- R16, R9: value 25121WF470 -> 25121WF101
- R24: footprint 04_MyFoot_Passive:R_2012Metric -> 04_MyFoot_Passive:R_3216Metric
- R27: value W4F7502 -> W4F7502(95k)
- R3: value AR06CTC0500 -> AR06CTC0500(220R)
- R34: value W4F1002 -> W4F1002(5k)
- T1: value TOROID_OUTPUT_OD20_T6T12 -> TOROID_OUTPUT_OD20_T6T12(T7:T24)
Connections:
- D9 pad 2: Net-(D9-A1) -> Net-(D9-A2)
- D9 pad 3: Net-(D9-common) -> GND
- J7 pad 2: Net-(D9-common) -> Net-(D9-A2)
- R40 pad 2: Net-(D9-common) -> Net-(D9-A2)
- SW2 pad 4: Net-(D9-common) -> Net-(D9-A2)
- U5 pad 7: Net-(D9-common) -> Net-(D9-A2)
Routing:
- net GND: track 1481.6 -> 1532.2 mm
- net Net-(D9-common): track 50.6 -> 0.00 mm
