File: kicad/ELSONIC/Multi_Mega_Main_V3/Multi_Mega_Main_V3.kicad_sch (KiCad schematic)
At the start: 196 parts, among them IC1 LM5005MHX_NOPB, J1 SMW250-02P, J10 DB25_Socket, J11 Conn_02x13_Odd_Even, J2 Screw_Terminal_01x06, J3 ARM_SWD_10, J4 Conn_01x06_HEADERPIN, J5 Conn_01x03, J6 Conn_02x10_Odd_Even, J7 SMW250-02P, J8 Conn_02x13_Odd_Even, J9 DB25_Pins, K1 G6A274, K2 PA1A_5V, K3 PA1A_5V, K4 G6A274, K5 PA1A_5V, K6 G6A274, K7 PA1A_5V, K8 PA1A_5V, K9 G6A274, Q1 STD25N10F7, Q2 STD25N10F7, SW1 TS-1088, SW2 DSHP02T, T1 TOROID_OUTPUT_OD20_T6T12, T2 TOROID_CT_OD16_T1T20, U1 AMS1117-3.3, U10 TLP185GB-S, U11 TLP185GB-S, U12 TLP185GB-S, U2 UCC21520DWR, U3 STM32G474RBT6, U4 INA190A3IDCKR, U5 MAX3485ESA, U6 TLP185GB-S, U7 ULN2003ADR, U8 ULN2003ADR, U9 TLP185GB-S, Y1 X49SM8M

Commit message: chore: sync remaining hardware design assets
Parts:
- removed J10: DB25_Socket, symbol Connector:DB25_Socket
- removed J11: Conn_02x13_Odd_Even, 02_MyFoot_Connectors:IDC-Header_2x13_P2.54mm_Latch_Vertical, symbol 02_MyLib_Connectors:Conn_02x13_Odd_Even
- removed J9: DB25_Pins, symbol Connector:DB25_Pins
- added IC2: L7987TR, 01_MyFoot_ICs:SOP65P640X120-17N, symbol 01_MyLib_ICs:L7987TR
- added L9: 33uH, 04_MyFoot_Passive:L_Radial_D10.0mm_P5.00mm, symbol 04_MyLib_Passive:Inductor
- added R52: W4F7502(200k), 04_MyFoot_Passive:R_3216Metric, symbol 04_MyLib_Passive:R
- added R53: 5K, 04_MyFoot_Passive:R_3216Metric, symbol 04_MyLib_Passive:R
- added R54: W4F9102, 04_MyFoot_Passive:R_3216Metric, symbol 04_MyLib_Passive:R
- added R55: W4F1002(5k), 04_MyFoot_Passive:R_3216Metric, symbol 04_MyLib_Passive:R
- added R56: 22K, 04_MyFoot_Passive:R_3216Metric, symbol 04_MyLib_Passive:R
- added R57, R58: W8J0103, 04_MyFoot_Passive:R_2012Metric, symbol 04_MyLib_Passive:R
- C42: value 1uF100V -> 0.1uF100V
- L2: value 3.9uH -> 4.7uH
- L4: value 1.5uH -> 1.0uH
- L6: value 2.7uH -> 2.2uH
- R12, R19: value 1812J103 -> 1812J222; LCSC C2933913 -> (none)
- R16, R9: value 25121WF470 -> 25121WF101; LCSC C474195 -> (none)
- R24: footprint 04_MyFoot_Passive:R_2012Metric -> 04_MyFoot_Passive:R_3216Metric
- R27: value W4F7502 -> W4F7502(95k)
- R3: value AR06CTC0500 -> AR06CTC0500(220R); LCSC C5266090 -> (none)
- R34: value W4F1002 -> W4F1002(5k)
- R4: LCSC C5266090 -> (none)
- T1: value TOROID_OUTPUT_OD20_T6T12 -> TOROID_OUTPUT_OD20_T6T12(T7:T24)
Connections:
- net ADC2_IN4: now also R54.1, R55.2
- net DAC1_OUT1: now also R56.2
- net GND: now also R55.1, R57.1, R58.1
- net GNDB: now also R53.1
- net INA: now also R57.2
- net INB: now also R58.2
- new net: IC2.9 (FB), R52.1, R53.2, R56.1
- new net: L9.2, R52.2, R54.2
- new net: IC2.13 (LX_1), IC2.14 (LX_2), L9.1
Other:
- note added: "10(ID)16(OD)SN-02HT CT 1:10T(2:15)"
- note removed: "10(ID)16(OD)SN-02HT CT 1:20T"
- moved on the sheet: C61, C62, D9, J7, R11, R13, R36, R37, R40, SW2, U5

Commit message: feat: update ultrasonic controller and board design
Connections:
- net GND: now also D9.3 (common)
- net at D9.1 (A1), J7.1, R36.1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: no longer D9.2 (A2)
- net at J7.2, R40.2, SW2.4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: now also D9.2 (A2); no longer D9.3 (common)
Changed lines of the file:
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@@
 	)
 	(junction
+		(at 469.9 299.72)
+		(diameter 0)
+		(color 0 0 0 0)
+	)
+	(junction
 		(at 403.86 135.89)
 		(diameter 0)
@@
 	)
 	(junction
-		(at 454.66 290.83)
-		(diameter 0)
-		(color 0 0 0 0)
-	)
-	(junction
 		(at 444.5 135.89)
 		(diameter 0)
@@
 	)
 	(junction
-		(at 462.28 285.75)
-		(diameter 0)
-		(color 0 0 0 0)
-	)
-	(junction
 		(at 548.64 101.6)
 		(diameter 0)
@@
 	(wire
 		(pts
-			(xy 488.95 299.72) (xy 454.66 299.72)
+			(xy 488.95 299.72) (xy 469.9 299.72)
 		)
 		(stroke
@@
 	(wire
 		(pts
-			(xy 462.28 298.45) (xy 462.28 285.75)
-		)
-		(stroke
-			(width 0)
-			(type default)
-		)
-	)
-	(wire
-		(pts
 			(xy 83.82 236.22) (xy 83.82 237.49)
 		)
@@
 	(wire
 		(pts
+			(xy 469.9 298.45) (xy 469.9 299.72)
+		)
+		(stroke
+			(width 0)
+			(type default)
+		)
+	)
+	(wire
+		(pts
 			(xy 424.18 290.83) (xy 412.75 290.83)
 		)
@@
 	(wire
 		(pts
+			(xy 466.09 289.56) (xy 462.28 289.56)
+		)
+		(stroke
+			(width 0)
+			(type default)
+		)
+	)
+	(wire
+		(pts
 			(xy 337.82 306.07) (xy 337.82 321.31)
 		)
@@
 	(wire
 		(pts
-			(xy 466.09 289.56) (xy 454.66 289.56)
-		)
-		(stroke
-			(width 0)
-			(type default)
-		)
-	)
-	(wire
-		(pts
 			(xy 303.53 167.64) (xy 309.88 167.64)
 		)
@@
 	(wire
 		(pts
+			(xy 462.28 289.56) (xy 462.28 292.1)
+		)
+		(stroke
+			(width 0)
+			(type default)
+		)
+	)
+	(wire
+		(pts
 			(xy 181.61 95.25) (xy 193.04 95.25)
 		)
@@
 	(wire
 		(pts
+			(xy 469.9 299.72) (xy 454.66 299.72)
+		)
+		(stroke
+			(width 0)
+			(type default)
+		)
+	)
+	(wire
+		(pts
 			(xy 389.89 90.17) (xy 389.89 85.09)
 		)
@@
 	(wire
 		(pts
-			(xy 454.66 289.56) (xy 454.66 290.83)
-		)
-		(stroke
-			(width 0)
-			(type default)
-		)
-	)
-	(wire
-		(pts
 			(xy 214.63 360.68) (xy 203.2 360.68)
 		)
@@
 	(wire
 		(pts
-			(xy 469.9 298.45) (xy 462.28 298.45)
-		)
-		(stroke
-			(width 0)
-			(type default)
-		)
-	)
-	(wire
-		(pts
 			(xy 496.57 41.91) (xy 496.57 49.53)
 		)
@@
 		(lib_id "Diode:SM712_SOT23")
 		(at 469.9 289.56 270)
-		(mirror x)
 		(unit 1)
 		(body_style 1)
@@
 		(dnp no)
 		(property "Reference" "D9"
-			(at 472.44 288.29 90)
+			(at 472.44 290.83 90)
 			(show_name no)
 			(do_not_autoplace no)
@@
 		)
 		(property "Value" "SM712-LF-T7"
-			(at 472.44 290.83 90)
+			(at 472.44 288.29 90)
 			(show_name no)
 			(do_not_autoplace no)
@@
 		)
 		(property "Datasheet" ""
-			(at 469.9 293.37 0)
+			(at 469.9 285.75 0)
 			(hide yes)
 			(show_name no)
@@
 					(unit 1)
 				)
+			)
+		)
+	)
+	(symbol
+		(lib_id "power:GND")
+		(at 462.28 292.1 0)
+		(unit 1)
+		(body_style 1)
+		(exclude_from_sim no)
+		(in_bom yes)
+		(on_board yes)
+		(in_pos_files yes)
+		(dnp no)
+		(property "Reference" "#PWR0150"
+			(at 462.28 298.45 0)
+			(hide yes)
+			(show_name no)
+			(do_not_autoplace no)
+			(effects
+				(font
+					(size 1.27 1.27)
+				)
+			)
+		)
+		(property "Value" "GND"
+			(at 465.836 293.878 0)
+			(show_name no)
+			(do_not_autoplace no)
+			(effects
+				(font
+					(size 1.27 1.27)
+				)
+			)
+		)
+		(property "Footprint" ""
+			(at 462.28 292.1 0)
+			(hide yes)
+			(show_name no)
+			(do_not_autoplace no)
+			(effects
+				(font
+					(size 1.27 1.27)
+				)
+			)
+		)
+		(property "Datasheet" ""
+			(at 462.28 292.1 0)
+			(hide yes)
+			(show_name no)
+			(do_not_autoplace no)
+			(effects
+				(font
+					(size 1.27 1.27)
+				)
+			)
+		)
+		(property "Description" "Power symbol creates a global label with name \"GND\" , ground"
+			(at 462.28 292.1 0)
+			(hide yes)
+			(show_name no)
+			(do_not_autoplace no)
+			(effects
+				(font
+					(size 1.27 1.27)
+				)
+			)
+		)
+		(pin "1"
+		)
+		(instances
+			(project "Multi_Mega_Main_V3"
+				(path "/846747d2-d9a3-4232-803f-01fc97424ea2"
+					(reference "#PWR0150")
+					(unit 1)
+				)
