File: kicad/ELSONIC/POWER_BD_SV6/POWER_BD_SV6.kicad_sch (KiCad schematic)
At the start: 102 parts, among them J2 SMW250-06P, J3 SMW250-02P, T2 EER28, U1 KP22315WGA, U2 EL354N, U3 TLP785(GB-TP6F), U4 ATTINY85-20PU_1, U5 MOC3021SM, U6 LM7805_TO220

Commit message: feat: update ultrasonic controller and board design
Parts:
- C11, C13: LCSC C76663 -> C3908730
Changed lines of the file:
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@@
 			)
 		)
-		(property "LCSC" "C76663"
+		(property "LCSC" "C3908730 "
 			(at 152.4 222.25 0)
 			(hide yes)
@@
 			)
 		)
-		(property "LCSC" "C76663"
+		(property "LCSC" "C3908730 "
 			(at 162.56 222.25 0)
 			(hide yes)
