File: kicad/ELSONIC/U-SONIC_Main_Stm_V1/U-SONIC_Main_Stm_V1.kicad_sch (KiCad schematic)
At the start: 226 parts, among them J1 SMW250-02P, J2 Screw_Terminal_01x06, J3 ARM_SWD_10, J4 Conn_01x06_HEADERPIN, J5 Conn_01x03, J6 SMW250-02P, J7 SMW250-02P, J8 Conn_02x13_Odd_Even, J9 SMW250-02P, K1 G6A274, K2 PA1A_5V, K3 PA1A_5V, Q1 STD25N10F7, Q10 KRC105S, Q2 STD25N10F7, Q3 IRF7341PBF, Q4 IRF7341PBF, Q5 IRF7341PBF, Q6 IRFP460PbF, Q7 IRFP460PbF, Q8 KRC105S, Q9 KRC105S, SW1 TS-1088, SW2 DSHP02T, T1 TOROID_OUTPUT_OD20_T6T12(T7:T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, T2 TOROID_CT_OD16_T1T20, U1 AMS1117-3.3, U10 TLP185GB-S, U11 TLP185GB-S, U12 TLP185GB-S, U13 IR2104, U14 IR2104, U15 74HCT04, U2 UCC21520DWR, U3 STM32G474RBT6, U4 INA190A3IDCKR, U5 MAX3485ESA, U6 TLP185GB-S, U9 TLP185GB-S, Y1 X49SM8M

Commit message: feat: update ultrasonic controller and board design
Parts:
- removed BZ1: SF1205A, 03_MyFoot_Active:Buzzer_12x9.5RM7.6, symbol Device:Buzzer
- removed C1, C16, C30, C33, C52, C53, C62, C64, C66, C7, C80, C81, C9: CL21B104K, 04_MyFoot_Passive:C_2012Metric, symbol 04_MyLib_Passive:C_Small
- removed C10, C2, C31, C34: 10UF25V67RV, 04_MyFoot_Passive:CP_Elec_4x5.4, symbol 04_MyLib_Passive:C_Pol
- removed C18: CG100J, 04_MyFoot_Passive:C_3216Metric, symbol 04_MyLib_Passive:C
- removed C20: CL21B475K, 04_MyFoot_Passive:C_2012Metric, symbol 04_MyLib_Passive:C_Small
- removed C24, C65: CL31B106K, 04_MyFoot_Passive:C_3216Metric, symbol 04_MyLib_Passive:C_Small
- removed C25: 0.1uF100V, 04_MyFoot_Passive:C_Rect_W7.0mm_P15.00mm, symbol 04_MyLib_Passive:C_Small
- removed C26: 10UF100V67RV, 04_MyFoot_Passive:CP_Elec_6.3x7.7, symbol 04_MyLib_Passive:C_Pol
- removed C27: 1000UF63V, 04_MyFoot_Passive:CP_Radial_D16.0mm_P7.50mm, symbol 04_MyLib_Passive:C_Pol
- removed C29, C8: 47UF50V67RV, 04_MyFoot_Passive:CP_Elec_6.3x7.7, symbol 04_MyLib_Passive:C_Pol
- removed C36, C41, C42: 0.1uF100V, 04_MyFoot_Passive:C_Rect_W7.0mm_P15.00mm, symbol 04_MyLib_Passive:C
- removed C43, C44: CL31B104K, 04_MyFoot_Passive:C_3216Metric, symbol 04_MyLib_Passive:C
- removed C46: 1206B223K101NT, 04_MyFoot_Passive:C_3216Metric, symbol 04_MyLib_Passive:C
- removed C49, C57: 1206CG331J101NT, 04_MyFoot_Passive:C_3216Metric, symbol 04_MyLib_Passive:C
- removed C50: 220UF50V67RV, 04_MyFoot_Passive:CP_Elec_10x10.5, symbol 04_MyLib_Passive:C_Pol
- removed C51, C73: CL31A106K, 04_MyFoot_Passive:C_3216Metric, symbol 04_MyLib_Passive:C
- removed C55: 1206CG102J101NT, 04_MyFoot_Passive:C_3216Metric, symbol 04_MyLib_Passive:C
- removed C58: 1206B103K, 04_MyFoot_Passive:C_3216Metric, symbol 04_MyLib_Passive:C
- removed C61, C63: CL31B105K, 04_MyFoot_Passive:C_3216Metric, symbol 04_MyLib_Passive:C_Small
- removed C67, C68, C69, C70, C71: CL21B472K, 04_MyFoot_Passive:C_2012Metric, symbol 04_MyLib_Passive:C_Small
- removed C74, C75: 2A103, 04_MyFoot_Passive:C_3216Metric, symbol 04_MyLib_Passive:C
- removed C76, C77: MF475, 04_MyFoot_Passive:C_3216Metric, symbol 04_MyLib_Passive:C
- removed C78: MLCC105, 04_MyFoot_Passive:C_3216Metric, symbol 04_MyLib_Passive:C
- removed C79: CL31B475K, 04_MyFoot_Passive:C_3216Metric, symbol 04_MyLib_Passive:C_Small
- removed D1: BAV99, 03_MyFoot_Active:SOT-23, symbol 03_MyLib_Active:BAV99
- removed D17, D18: MM3Z3V6, 03_MyFoot_Active:D_SOD-323_HandSoldering, symbol 03_MyLib_Active:MM3Z3V6
- removed D19, D2, D20, D3: SS24B, 03_MyFoot_Active:D_SMB, symbol 03_MyLib_Active:SS24B
- removed D21, D22: US1G, Diode_SMD:D_SMA, symbol Diode:US1G
- removed D4: BAT54WSQ-7, 03_MyFoot_Active:D_SOD-323_HandSoldering, symbol Diode:RF01VM2S
- removed D6: B3100-13-F, 03_MyFoot_Active:B3100_13_F, symbol 03_MyLib_Active:B3100-13-F
- removed D7: LL4148, 03_MyFoot_Active:LL4148_MELF, symbol 03_MyLib_Active:LL4148
- removed D9: SM712-LF-T7, Package_TO_SOT_SMD:SOT-23, symbol Diode:SM712_SOT23
- removed DCDC1, DCDC2: MUS2415N, 05_MyFoot_Others:MUS2415N, symbol 05_MyLib_Others:MUS2415N
- removed FC1, FC2: 470UF63V, 04_MyFoot_Passive:CP_Radial_D12.5mm_P5.00mm, symbol 04_MyLib_Passive:C_Pol
- removed H3, H4: MountingHole, 06_MyFoot_Mechanical:MTHole_3.5mm, symbol 06_MyLib_Mechanical:MountingHole
- removed J1, J7: SMW250-02P, 02_MyFoot_Connectors:SMW250_02P, symbol 02_MyLib_Connectors:SMW250-02P
- removed J2: Screw_Terminal_01x06, 02_MyFoot_Connectors:TB_P5.00mm_6P, symbol 06_MyLib_Mechanical:Screw_Terminal_01x06
- removed J4: Conn_01x06_HEADERPIN, 02_MyFoot_Connectors:PinHeader_1x06_P2.54mm_Vertical, symbol 02_MyLib_Connectors:Conn_01x06_HEADERPIN
- removed J5: Conn_01x03, 02_MyFoot_Connectors:PinHeader_1x03_P2.54mm_Vertical, symbol 02_MyLib_Connectors:Conn_01x03
- removed J6, J9: SMW250-02P, SMW25002, symbol 02_MyLib_Connectors:SMW250-02P
- removed J8: Conn_02x13_Odd_Even, 02_MyFoot_Connectors:IDC-Header_2x13_P2.54mm_Latch_Vertical, symbol 02_MyLib_Connectors:Conn_02x13_Odd_Even
- removed K1: G6A274, 06_MyFoot_Mechanical:G6A274PST15USDC12, symbol 06_MyLib_Mechanical:G6A274
- removed K2, K3: PA1A_5V, 06_MyFoot_Mechanical:PA1A5V, symbol 06_MyLib_Mechanical:PA1A_5V
- removed L1: 3.3uH, 04_MyFoot_Passive:L_Radial_D10.0mm_P5.00mm, symbol 04_MyLib_Passive:Inductor
- removed L2: 4.7uH, 04_MyFoot_Passive:L_Radial_D10.0mm_P5.00mm, symbol 04_MyLib_Passive:Inductor
- removed L3: 33uH, 04_MyFoot_Passive:L_Radial_D10.0mm_P5.00mm, symbol 04_MyLib_Passive:Inductor
- removed LCD1: LC1602A, 06_MyFoot_Mechanical:LC1602A, symbol 05_MyLib_Others:LC1602A
- removed Q1, Q2: STD25N10F7, Package_TO_SOT_SMD:TO-252-2, symbol 03_MyLib_Active:STD7N10F7
- removed Q10: KRC105S, 03_MyFoot_Active:SOT-23_KRC105S, symbol 03_MyLib_Active:KRC105S
- removed Q3, Q4, Q5: IRF7341PBF, Package_SO:SOIC-8_3.9x4.9mm_P1.27mm, symbol 03_MyLib_Active:IRF7341PBF
- removed Q6, Q7: IRFP460PbF, Package_TO_SOT_THT:TO-247-3_Vertical, symbol Transistor_FET:IRFP4668PbF
- removed R10: 15K/3W, 04_MyFoot_Passive:R_Axial_2W_P20.32mm, symbol 04_MyLib_Passive:R
- removed R3: AR06CTC0500, 04_MyFoot_Passive:R_3216Metric, symbol 04_MyLib_Passive:R
- removed R32, R54: W4J0100, 04_MyFoot_Passive:R_3216Metric, symbol 04_MyLib_Passive:R
- removed R38, R41: W4J0472, 04_MyFoot_Passive:R_3216Metric, symbol 04_MyLib_Passive:R
- removed R50: W4J0102, 04_MyFoot_Passive:R_3216Metric, symbol 04_MyLib_Passive:R
- removed R51: W4F0000, 04_MyFoot_Passive:R_3216Metric, symbol 04_MyLib_Passive:R
- removed R53, R55, R56: 0805FR-0747RL, 04_MyFoot_Passive:R_2012Metric, symbol 04_MyLib_Passive:R
- removed R57: 750ohms_1W, 04_MyFoot_Passive:R_2512_6332Metric, symbol 04_MyLib_Passive:R
- removed R58, R63: 30ohms_1/2W, 04_MyFoot_Passive:R_2512_6332Metric, symbol 04_MyLib_Passive:R
- removed R59, R62: 220ohms_1W, 04_MyFoot_Passive:R_2512_6332Metric, symbol 04_MyLib_Passive:R
- removed R60, R61: 1kohms_1W, 04_MyFoot_Passive:R_2512_6332Metric, symbol 04_MyLib_Passive:R
- removed R64, R65: 33kohms_3W, 04_MyFoot_Passive:R_2512_6332Metric, symbol 04_MyLib_Passive:R
- removed R66, R67: 0805FR-0747RL(4.7R), 04_MyFoot_Passive:R_2012Metric, symbol 04_MyLib_Passive:R
- removed R68: W4J0470, 04_MyFoot_Passive:R_3216Metric, symbol 04_MyLib_Passive:R
- removed R74: W4J0220, 04_MyFoot_Passive:R_3216Metric, symbol 04_MyLib_Passive:R
- removed SW1: TS-1088, 06_MyFoot_Mechanical:SW_SPST_TS-1088-xR025, symbol Switch:SW_Push
- removed SW2: DSHP02T, 06_MyFoot_Mechanical:CHS-02B_W7.62mm_P1.27mm, symbol Switch:SW_DIP_x02
- removed T1: TOROID_OUTPUT_OD20_T6T12(T7:T24), 04_MyFoot_Passive:Toroid_OD20mm_ID10-T6T12, symbol 04_MyLib_Passive:TOROID_OUTPUT_OD20_T6T12
- removed T2: TOROID_CT_OD16_T1T20, 04_MyFoot_Passive:Toroid_OD16mm_ID9.6-T1T20, symbol 04_MyLib_Passive:TOROID_CT_OD16_T1T20
- removed TR2: EI2218_TAP, symbol 04_MyLib_Passive:EI2218_TAP
- removed TR3: OUTPUT-TRANS, Transformer_THT:Transformer_Breve_TEZ-28x33, symbol Transformer:TEZ1.5-D-1
- removed TS1, TS2, TS3, TS4: TS1103D, 06_MyFoot_Mechanical:SW_PUSH-12mm, symbol 06_MyLib_Mechanical:TS1103D
- removed U10, U11, U12, U6, U9: TLP185GB-S, 01_MyFoot_ICs:SOIC-4_4.55x3.7mm_P2.54mm, symbol Isolator:TLP185
- removed U13, U14: IR2104, symbol 01_MyLib_ICs:IR2104
- removed U15: 74HCT04, symbol 01_MyLib_ICs:74HCT04
- removed U2: UCC21520DWR, 01_MyFoot_ICs:SOIC-16W_7.5x10.3mm_P1.27mm, symbol 01_MyLib_ICs:UCC21520DW
- removed U3: STM32G474RBT6, Package_QFP:LQFP-64_10x10mm_P0.5mm, symbol 00_MyLib_MCU:STM32G474RBT6
- removed U4: INA190A3IDCKR, Package_TO_SOT_SMD:SOT-363_SC-70-6, symbol 01_MyLib_ICs:INA190A3
- removed U5: MAX3485ESA, 01_MyFoot_ICs:SOIC-8_3.9x4.9mm_P1.27mm, symbol 01_MyLib_ICs:MAX3485ESA
- added C11: CL31B475K, 04_MyFoot_Passive:C_3216Metric, symbol 04_MyLib_Passive:C_Small
- added C13, C15, C24, C36: 10UF25V67RV, 04_MyFoot_Passive:CP_Elec_4x5.4, symbol 04_MyLib_Passive:C_Pol
- added C14, C21, C22: CL31B105K, 04_MyFoot_Passive:C_3216Metric, symbol 04_MyLib_Passive:C
- added C18, C26: 22pF, 04_MyFoot_Passive:C_3216Metric, symbol 04_MyLib_Passive:C_Small
- added C23, C25, C27, C29, C35, C9: CL31B104K, 04_MyFoot_Passive:C_3216Metric, symbol 04_MyLib_Passive:C
- added C40, C46, C47: CL21B104K, 04_MyFoot_Passive:C_2012Metric, symbol 04_MyLib_Passive:C_Small
- added C45: CL31B105K, 04_MyFoot_Passive:C_3216Metric, symbol 04_MyLib_Passive:C_Small
- added D1, D6: UF4007, 03_MyFoot_Active:D_SMA, symbol 03_MyLib_Active:UF4007
- added D11, D12, D3, D7, D9: BAT54WSQ-7, 03_MyFoot_Active:D_SOD-323_HandSoldering, symbol Diode:RF01VM2S
- added D13, D2, D4, D8: LL4148, 03_MyFoot_Active:LL4148_MELF, symbol 03_MyLib_Active:LL4148
- added H1, H3: MountingHole_Pad, 06_MyFoot_Mechanical:MTHole_3.5mm_6.8mmPad_GND, symbol 06_MyLib_Mechanical:MountingHole_Pad
- added J2, J7: SMW250-04P, 02_MyFoot_Connectors:SMW250_04P, symbol 02_MyLib_Connectors:SMW250-04P
- added J3: SMW250-02P, 02_MyFoot_Connectors:SMW250_02P, symbol 02_MyLib_Connectors:SMW250-02P
- added J4: SW_BD, 05_MyFoot_Others:SW_BD, symbol 05_MyLib_Others:SW_BD
- added J5: SMW250-06P, 02_MyFoot_Connectors:SMW250_06P, symbol 02_MyLib_Connectors:SMW250-06P
- added J6: SMW250-08P, 02_MyFoot_Connectors:SMW250_08P, symbol 02_MyLib_Connectors:SMW250-08P
- added J8: RS485_BD, 02_MyFoot_Connectors:IDC-Header_2x05_P2.54mm_Vertical, symbol 02_MyLib_Connectors:Conn_02x05_Odd_Even
- added K1, K2: HR92, 06_MyFoot_Mechanical:Relay_SPDT_HsinDa_Y14, symbol 06_MyLib_Mechanical:HR92
- added LCD1: LC1622, 06_MyFoot_Mechanical:LC1622_1, symbol 05_MyLib_Others:LC1622
- added LED1, LED2: LED_SMD_KT_0805R, 03_MyFoot_Active:LED_2012Metric, symbol 03_MyLib_Active:LED_SMD_KT_0805R
- added LS1: MLT-8530, 03_MyFoot_Active:MLT8530, symbol 03_MyLib_Active:MLT-8530
- added OP_1, OP_2, OP_3, OP_4: TAP_250, 02_MyFoot_Connectors:TAP_250, symbol 02_MyLib_Connectors:TAP_250
- added Q1, Q2: IRF7351, 01_MyFoot_ICs:SOIC-8_3.9x4.9mm_P1.27mm, symbol 03_MyLib_Active:IRF7351
- added Q4: KRC105S, 03_MyFoot_Active:SOT-23_KRC105S, symbol 03_MyLib_Active:KRC105S
- added Q5: 2SC5343, 03_MyFoot_Active:SOT-23, symbol 03_MyLib_Active:2SC5343
- added R11: WR08X1000FTL, 04_MyFoot_Passive:R_2012Metric, symbol 04_MyLib_Passive:R
- added R23, R24: 1K, 04_MyFoot_Passive:R_3216Metric, symbol 04_MyLib_Passive:R
- added R29: RS-06K47R, 04_MyFoot_Passive:R_3216Metric, symbol 04_MyLib_Passive:R
- added T1: SCT-17P, 04_MyFoot_Passive:SCT-17P, symbol 04_MyLib_Passive:SCT-17P
- added TP1, TP10, TP11, TP12, TP2, TP3, TP4, TP5, TP6, TP7, TP8, TP9: TPOINT, 05_MyFoot_Others:TP, symbol 05_MyLib_Others:TPOINT
- added U1: 74AHCT125, 01_MyFoot_ICs:SOIC-14_3.9x8.7mm_P1.27mm, symbol 01_MyLib_ICs:74AHCT125
- added U2, U4: IR2104, 01_MyFoot_ICs:SOIC-8_3.9x4.9mm_P1.27mm, symbol 01_MyLib_ICs:IR2104
- added U3: STM32G474CBT6, Package_QFP:LQFP-48_7x7mm_P0.5mm, symbol 00_MyLib_MCU:STM32G474C_B-C-E_Tx
- added U5: 74HCT574PWR, 01_MyFoot_ICs:TSSOP-20_4.4x6.5mm_P0.65mm, symbol 01_MyLib_ICs:74HCT574
- C12: value CG100J -> CL31B105K; LCSC C1883 -> C1848
- C28: value CL21B104K -> CL31B475K; footprint 04_MyFoot_Passive:C_2012Metric -> 04_MyFoot_Passive:C_3216Metric; LCSC C1711 -> C1872
- C37, C38: LCSC C1945 -> C24497
- C8: renamed from C72; value CL31A106K -> CL31B105K; LCSC C13585 -> C1848
- D10: LCSC C84062 -> C68883
- R12: value 1812J103 -> RS-06K103JT; footprint 04_MyFoot_Passive:R_4532Metric -> 04_MyFoot_Passive:R_3216Metric; LCSC C2933913 -> C118075
- R14: value W8J0103 -> 100K/1W; footprint 04_MyFoot_Passive:R_2012Metric -> 04_MyFoot_Passive:R_6332Metric; LCSC C25612 -> C52842
- R15: value 0805FR-07100K -> FRC1206F2400TS; footprint 04_MyFoot_Passive:R_2012Metric -> 04_MyFoot_Passive:R_3216Metric; LCSC C96346 -> C2933649
- R16: value 25121WF470 -> WR08X1002FTL; footprint 04_MyFoot_Passive:R_6332Metric -> 04_MyFoot_Passive:R_2012Metric; LCSC C474195 -> C108451
- R17: value 15K/3W -> 10K; footprint 04_MyFoot_Passive:R_Axial_2W_P20.32mm -> 04_MyFoot_Passive:R_3216Metric; LCSC (none) -> C183193
- R18: value 22K/3W -> 100K/1W; footprint 04_MyFoot_Passive:R_Axial_2W_P20.32mm -> 04_MyFoot_Passive:R_6332Metric; LCSC (none) -> C52842
- R19: value 1812J103 -> RS-06K22R; footprint 04_MyFoot_Passive:R_4532Metric -> 04_MyFoot_Passive:R_3216Metric; LCSC C2933913 -> C140034
- R20: value W4F1002 -> WR08X1002FTL; footprint 04_MyFoot_Passive:R_3216Metric -> 04_MyFoot_Passive:R_2012Metric; LCSC C17902 -> C108451
- R21: value W4F1002 -> RS-06K103JT; LCSC C17902 -> C118075
- R22: value 0805FR-0733RL -> WR08X1002FTL; LCSC C126353 -> C108451
- R25: value W8J0103 -> RS-06K22R; footprint 04_MyFoot_Passive:R_2012Metric -> 04_MyFoot_Passive:R_3216Metric; LCSC C25612 -> C140034
- R26: value FRL2512FR047TS-47mohm -> RS-06K103JT; footprint 04_MyFoot_Passive:R_2512_6332Metric -> 04_MyFoot_Passive:R_3216Metric; LCSC C7467449 -> C118075
- R27: value W4F7502(120k) -> RS-05K472JT; footprint 04_MyFoot_Passive:R_3216Metric -> 04_MyFoot_Passive:R_2012Metric; LCSC C17986 -> C115310
- R28: value W4F9102 -> WR08X1002FTL; footprint 04_MyFoot_Passive:R_3216Metric -> 04_MyFoot_Passive:R_2012Metric; LCSC C17981 -> C108451
- R3: renamed from R52; value 0805FR-0747RL -> RS-06K22R; footprint 04_MyFoot_Passive:R_2012Metric -> 04_MyFoot_Passive:R_3216Metric; LCSC C114541 -> C140034
- R33: value W4F4991 -> FRC1206F2400TS; LCSC C57609 -> C2933649
- R34: value W4F1002(5k) -> 10K; LCSC C17902 -> C183193
- R35: value W4F8871 -> FRC1206F2400TS; LCSC C55354 -> C2933649
- R36: value W8J0431 -> 1K; footprint 04_MyFoot_Passive:R_2012Metric -> 04_MyFoot_Passive:R_3216Metric; LCSC C54672 -> C131398
- R37: value W4J0121 -> 10K; LCSC C25351 -> C183193
- R4: value AR06CTC0500 -> RS-06K103JT; LCSC C5266090 -> C118075
- R40: value W8J0431 -> RS-05K470JT; LCSC C54672 -> C139871
- R42, R44: value W8J0103 -> 0805W8J0202T5E; LCSC C25612 -> C1359
- R43: value W4J0472 -> 0805W8F1000T; footprint 04_MyFoot_Passive:R_3216Metric -> 04_MyFoot_Passive:R_2012Metric; LCSC C26043 -> C17408
- R45: value W4J0472 -> W8J0103; footprint 04_MyFoot_Passive:R_3216Metric -> 04_MyFoot_Passive:R_2012Metric; LCSC C26043 -> C25612
- R46: value W8J0103 -> RS-05K470JT; LCSC C25612 -> C139871
- R47: value W4J0472 -> RS-05K471JT; footprint 04_MyFoot_Passive:R_3216Metric -> 04_MyFoot_Passive:R_2012Metric; LCSC C26043 -> C119076
- R49: value W4J0102 -> RS-05K470JT; footprint 04_MyFoot_Passive:R_3216Metric -> 04_MyFoot_Passive:R_2012Metric; LCSC C1469 -> C139871
- R5: value W4F4700 -> 1K; LCSC C4502 -> C131398
- R6: value W4F4700 -> RS-06K22R; LCSC C4502 -> C140034
- R7: value W4F4700 -> 100K/1W; footprint 04_MyFoot_Passive:R_3216Metric -> 04_MyFoot_Passive:R_6332Metric; LCSC C4502 -> C52842
- R8: value W4F4700 -> FRC1206F2400TS; LCSC C4502 -> C2933649
- R9: value 25121WF470 -> 10K; footprint 04_MyFoot_Passive:R_6332Metric -> 04_MyFoot_Passive:R_3216Metric; LCSC C474195 -> C183193
- TR1: footprint Transformer_THT:Transformer_Breve_TEZ-22x24 -> 04_MyFoot_Passive:EI2218
- renumbered C11 to C1, C23 to C10, C32 to C16, C35 to C17, C39 to C19, C13 to C2, C40 to C20, C14 to C3, C82 to C30, C83 to C31, C84 to C32, C86 to C33, C88 to C34, C85 to C39, C15 to C4, C3 to C41, C4 to C42, C5 to C43, C6 to C44, C22 to C5, C19 to C6, C21 to C7, D23 to D14, D8 to D15, H1 to H4, J3 to J1, Q8 to Q3, Q9 to Q6, R2 to R1, R11 to R10, R1 to R2, R69 to R30, R71 to R31, R73 to R32, R70 to R38, U1 to U6
Connections:
- net BCD_BIT3_M is gone; now on net REMOTE: R46.1
- net GNDA is gone; now on net GND: R12.1
- net REMOTE_M is gone; now on net RUN_SW: R39.1
- net SENSOR_M is gone; now on net SWEEP_SW: R48.1
- net USART1_TX is gone; now on net /RE_RS485: R22.2
- net +12V: now also C12.2, C13.1, C14.2, C15.1, C21.2, D1.2 (A), D6.2 (A), J5.1, Q1.7 (D1), Q1.8 (D1), Q2.7 (D1), Q2.8 (D1), U2.1 (VCC), U4.1 (VCC)
- net +3.3V: now also D14.1 (K), R27.2, R28.2, R34.2, R45.2, R9.2, D11.1 (K), D3.1 (K), D7.1 (K), J6.8, LS1.2 (+LEAD), U3.1 (VBAT), U3.24 (VDD), U3.36 (VDD), U3.48 (VDD); no longer R36.2, R44.2, R46.2
- net +5V: now also C28.2, R44.2, C27.2, C29.2, D13.1 (K), J5.3, J8.1 (Pin_1), J8.2 (Pin_2), K1.3, K2.3, LCD1.2 (VDD), R29.2, U1.14 (VCC), U5.20 (VCC); no longer D10.1 (K)
- net 485BD_DETECT: now also R28.1, J8.8 (Pin_8), U3.40 (PB3)
- net ADC2_IN3: now also C38.2, R36.1, D11.2 (A), D12.1 (K), TP1.1 (Pin_1), U3.14 (PA6)
- net BZ_OUT: now also U3.13 (PA5)
- net CHA1: now also U3.30 (PA8)
- net CHA2: now also U3.31 (PA9)
- net DE_RS485: now also R20.2, J8.6 (Pin_6), U3.41 (PB4)
- net DOWN: now also C34.1, R32.1, J4.3 (Pin_3), U3.44 (PB7); no longer C39.1, R38.1
- net END_BZ: now also U3.3 (PC14)
- net GND: now also C37.1, C38.1, D5.2 (A), R16.1, R17.1, R22.1, R26.1, R37.1, C11.1, C13.2, C14.1, C15.2, C18.1, C21.1, C24.2, C25.1, C26.1, C27.1, C29.1, C35.1, C36.2, C40.2, C45.1, C46.2, C47.2, D12.2 (A), D9.2 (A), H1.1, H3.1, J4.5 (Pin_5), J4.6 (Pin_6), J4.7 (Pin_7), J4.8 (Pin_8), J5.2, J5.4, J6.1, J6.3, J6.5, J8.10 (Pin_10), LCD1.1 (VSS), LCD1.16 (LED(-)), LCD1.17, LCD1.18, LCD1.19, LCD1.20, LCD1.5 (R/W), LED2.2 (K), Q1.3 (S2), Q2.3 (S2), Q4.2 (E), Q5.2 (E), TP10.1 (Pin_1), TP2.1 (Pin_1), TP4.1 (Pin_1), TP6.1 (Pin_1), TP8.1 (Pin_1), U1.1, U1.10, U1.12, U1.4, U1.7 (GND), U2.4 (COM), U3.19 (VSSA), U3.23 (VSS), U3.35 (VSS), U3.47 (VSS), U4.4 (COM), U5.1 (OE), U5.10 (GND); no longer R14.1, R15.1, R21.1, R25.1, R34.1, R4.1, R40.1
- net GOING: now also Q4.1 (B), U3.2 (PC13)
- net INA: now also U1.2
- net INB: now also U1.5
- net LCD_D4: now also U3.26 (PB12), U5.4 (D2)
- net LCD_D5: now also U3.27 (PB13), U5.5 (D3)
- net LCD_D6: now also U3.28 (PB14), U5.6 (D4)
- net LCD_D7: now also U3.29 (PB15), U5.7 (D5)
- net LCD_E: now also U3.25 (PB11), U5.2 (D0)
- net LCD_RS: now also U3.22 (PB10), U5.3 (D1)
- net MODE: now also C39.1, R38.1, J4.4 (Pin_4), U3.43 (PB6); no longer C33.1, R31.1
- net NRST: now also U3.7 (PG10)
- net PWM_OUTPUT: now also R47.2, U3.15 (PA7)
- net PWM_VR: now also R43.1, C45.2, U3.17 (PB1)
- net REMOTE: now also R45.1, C46.1, U3.32 (PA10)
- net RTERM: now also J8.7 (Pin_7), U3.18 (PB2)
- net RUN_SW: now also R40.1, C40.1, U3.33 (PA11)
- net SONIC_ON: now also R11.1, U3.39 (PA15)
- net START_STOP: now also J4.1 (Pin_1), U3.46 (PB9)
- net SWCLK: now also U3.38 (PA14)
- net SWDIO: now also U3.37 (PA13)
- net SWEEP_SW: now also R49.1, C47.1, U3.34 (PA12)
- net UP: now also C33.1, R31.1, J4.2 (Pin_2), U3.45 (PB8); no longer C34.1, R32.1
- net USART2_RX: now also R27.1, U1.11, U3.11 (PA3)
- net USART2_TX: now also U1.9, U3.10 (PA2)
- net /RE_RS485: now also J8.4 (Pin_4), U3.42 (PB5)
- net at D14.2 (A), Q3.3 (C): now also LS1.3 (-LEAD)
- net at R16.2: now also R11.2, U2.3 (~{SD}), U4.3 (~{SD})
- net at R19.2: now also R21.2, D8.2 (A), Q2.2 (G1); no longer R16.1
- net at R40.2: now also J6.7
- net ADC1_IN2_COMP1: now reaches D5.1 (K)
- net ADC1_IN2_COMP1: now also R5.1, C18.2, D3.2 (A), TP3.1 (Pin_1), U3.9 (PA1); no longer R21.2
- net at D10.2 (A): now also R25.2, R26.2, Q2.4 (G2)
- net at C8.2: now also C9.2, D1.1 (K), U2.8 (VB)
- net at R37.2: now also C37.2, R33.1, R34.1, R35.1, C36.1, J3.2
- net at C17.2, Y1.1: now also U3.6 (PF1)
- net at R47.1: now also Q5.1 (B)
- net at R5.2: now also R15.2, R8.2, T1.3; no longer R6.2
- net at C8.1: now also R4.1, TR1.2, C9.1, Q1.1 (S1), Q1.5 (D2), Q1.6 (D2), TP11.1 (Pin_1), U2.6 (VS)
- net at R3.1: now also D2.1 (K), U2.7 (HO)
- net at R9.1: now also R15.1, R17.2, R8.1, C24.1, C25.2, R24.1, T1.4; no longer R12.2
- net at R3.2: now also R4.2, D2.2 (A), Q1.2 (G1)
- net at RV1.2: now also C35.2, LCD1.3 (VO)
- net at C16.2, Y1.2: now also U3.5 (PF0)
- net at C10.2, C6.2, FB1.2: now also C11.2, U3.20 (VREF+), U3.21 (VDDA)
- net at D15.2 (A), Q6.3 (C): now also K2.4
- net at R14.2: now also R7.1
- net at TR1.4: now also R21.1, C22.1, C23.1, Q2.1 (S1), Q2.5 (D2), Q2.6 (D2), TP12.1 (Pin_1), U4.6 (VS)
- net at TR1.10: now also J2.4
- net at TR1.6: now also J2.1
- net at TR1.7: now also J2.2
- net at TR1.9: now also J2.3
- removed net +24V: C28.2, R43.2, R45.2, R47.2
- net +VBUS: no longer names the net of R18.2
- net +VBUS: now also R14.1; no longer R26.1
- net ADC1_IN1: no longer names the net of R49.2
- net ADC1_IN1: now also J6.2
- removed net ADC2_IN4: R28.1, R34.2
- net BCD_BIT1_M: no longer names the net of R42.1
- net BCD_BIT1_M: now also LED1.1 (A)
- net BCD_BIT2_M: no longer names the net of R44.1
- net BCD_BIT2_M: now also LED2.1 (A)
- net DAC1_OUT1: no longer names the net of R35.2
- net DAC1_OUT1: now also R33.2, R36.2, J3.1
- removed net GNDB: R17.1, R18.1, R19.1, R33.1
- new net: C22.2, C23.2, D6.1 (K), U4.8 (VB)
- new net: TP9.1 (Pin_1), U1.6, U4.2 (IN)
- new net: J6.6, R46.2
- new net: TP7.1 (Pin_1), U1.3, U2.2 (IN)
- new net: D10.1 (K), R25.1, U4.5 (LO)
- new net: D4.2 (A), Q1.4 (G2), R12.2, R6.2
- new net: J6.4, R43.2
- new net: D13.2 (A), K1.4, Q4.3 (C)
- new net: D4.1 (K), R6.1, U2.5 (LO)
- new net: D8.1 (K), R19.1, U4.7 (HO)
- new net: R18.1, R23.1, R24.2
- new net: OP_3.1 (Pin_1), OP_3.2 (Pin_2), OP_4.1 (Pin_1), OP_4.2 (Pin_2)
- new net: J7.2, K1.1
- new net: J7.1, K1.5, K1.6
- new net: J7.3, K2.5, K2.6
- new net: J7.4, K2.1
- new net: LCD1.11 (D4), U5.17 (Q2)
- new net: LCD1.12 (D5), U5.16 (Q3)
- new net: LCD1.13 (D6), U5.15 (Q4)
- new net: LCD1.14 (D7), U5.14 (Q5)
- new net: LCD1.15 (LED(+)), R29.1
- new net: LCD1.4 (RS), U5.19 (Q0)
- new net: LCD1.6 (E), U5.18 (Q1)
- new net 50V_550V_15kHz_128kHz: OP_1.1 (Pin_1), OP_1.2 (Pin_2), OP_2.1 (Pin_1), OP_2.2 (Pin_2), R7.2
- new net ADC1_IN1_COMP3: C26.2, D7.2 (A), D9.1 (K), R23.2, TP5.1 (Pin_1), U3.8 (PA0)
- new net CLK_LCD: U3.16 (PB0), U5.11 (Cp)
- new net MAX485_RX: J8.3 (Pin_3), U1.13
- new net MAX485_TX: J8.5 (Pin_5), U1.8
- new net PWM_COLLECTOR: J5.6, Q5.3 (C)
- new net RUN_LED: LED1.2 (K), U3.12 (PA4)
- new net SPARE: J8.9 (Pin_9), U3.4 (PC15)
- no-connect marks 24 -> 17
Other:
- note added: "1.618V"
- note added: "1.623V"
- note added: "10(ID)16(OD)CT 1:1000T"
- note added: "10(ID)16(OD)SN-02HT CT 1:1000T"
- note added: "PA2 TX ── 74AHCT02 ── MAX485 DI PA3 RX ◀─ 3.3V LVC 버퍼 ◀─ MAX485 RO PB4 DE ────────────────── MAX485 DE PB5 /RE ───────────────── MAX485 /RE PB2 RTERM ──────────────── KRC105M PB3 DETECT ◀────────────── SPARE1"
- note added: "PA2 TX ── 74AHCT125 ── MAX485 DI PA3 RX ◀─ 3.3V LVC 버퍼 ◀─ MAX485 RO PB4 DE ────────────────── MAX485 DE PB5 /RE ───────────────── MAX485 /RE PB2 RTERM ──────────────── KRC105M PB3 DETECT ◀────────────── SPARE1"
- note removed: "10(ID)16(OD)SN-02HT CT 1:20T(2:15)"
- note removed: "PL-F2 OUTPUT TRANS 20(OD)10(ID) 6T:12T LITZ 0.2mm ENAMEL"
- moved on the sheet: C1, C10, C16, C17, C19, C2, C20, C3, C30, C31, C32, C33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
