File: kicad/ELSONIC/U-SONIC_Main_Stm_V1/U-SONIC_Main_Stm_V1.kicad_sch (KiCad schematic)
At the start: 161 parts, among them J1 ARM_SWD_10, J2 SMW250-04P, J3 SMW250-02P, J4 SW_BD, J5 SMW250-06P, J6 SMW250-08P, J7 SMW250-04P, J8 RS485_BD, K1 HR92, K2 HR92, Q1 IRF7351, Q2 IRF7351, Q3 KRC105S, Q4 KRC105S, Q5 2SC5343, Q6 KRC105S, T1 SCT-17P, U1 74AHCT125, U2 IR2104, U3 STM32G474CBT6, U4 IR2104, U5 74HCT574PWR, U6 AMS1117-3.3, Y1 X49SM8M

Commit message: feat: update STM32 firmware, docs, and board design
Co-authored-by: Copilot <223556219+Copilot@users.noreply.github.com>
Other:
- note added: "100ohms로 변경 필요"
- moved on the sheet: J8, R27, R28, U1C, U1D
